File: Projets/Station_meteo/PCB/V0_Prototype/Modules/Interfaces.kicad_sch (KiCad schematic)
At the start: 3 parts, among them J31 Wind_Direction, J32 Water_Level

Commit message: Update PCB
Parts:
- removed C31: 100nF, Capacitor_SMD:C_0603_1608Metric, symbol Device:C
- removed J31: Wind_Direction, Connector_Phoenix_MSTB:PhoenixContact_MSTBA_2,5_2-G-5,08_1x02_P5.08mm_Horizontal, symbol Connector:Screw_Terminal_01x02
- added J35: Screw_Terminal_01x03, Connector_Phoenix_MSTB:PhoenixContact_MSTBA_2,5_3-G-5,08_1x03_P5.08mm_Horizontal, symbol Connector:Screw_Terminal_01x03
- added R21: 100k, Resistor_SMD:R_0603_1608Metric, symbol Device:R
Connections:
- net +3.3V: now also J35.1 (Pin_1), R21.1
- net GND: now also J32.2 (Pin_2), J35.3 (Pin_3)
- net Water_Level: now reaches J32.1 (Pin_1)
- net Water_Level: now also R21.2
- new net Direction: J35.2 (Pin_2)
Changed lines of the file:
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@@
 		(rev "1.0")
 	)
-	(bus_entry
-		(at 62.23 63.5)
-		(size -2.54 2.54)
-		(stroke
-			(width 0)
-			(type default)
-		)
-	)
-	(bus_entry
-		(at 62.23 60.96)
-		(size -2.54 2.54)
-		(stroke
-			(width 0)
-			(type default)
-		)
-	)
-	(bus
-		(pts
-			(xy 59.69 69.85) (xy 59.69 66.04)
-		)
-		(stroke
-			(width 0)
-			(type default)
-		)
-	)
-	(wire
-		(pts
-			(xy 82.55 43.18) (xy 82.55 44.45)
-		)
-		(stroke
-			(width 0)
-			(type default)
-		)
-	)
-	(bus
-		(pts
-			(xy 58.42 69.85) (xy 59.69 69.85)
+	(junction
+		(at 121.92 66.04)
+		(diameter 0)
+		(color 0 0 0 0)
+	)
+	(wire
+		(pts
+			(xy 118.11 66.04) (xy 121.92 66.04)
+		)
+		(stroke
+			(width 0)
+			(type default)
+		)
+	)
+	(wire
+		(pts
+			(xy 120.65 68.58) (xy 120.65 71.12)
+		)
+		(stroke
+			(width 0)
+			(type default)
+		)
+	)
+	(wire
+		(pts
+			(xy 121.92 44.45) (xy 125.73 44.45)
+		)
+		(stroke
+			(width 0)
+			(type default)
+		)
+	)
+	(wire
+		(pts
+			(xy 121.92 55.88) (xy 121.92 58.42)
 		)
 		(stroke
@@
 	(wire
 		(pts
-			(xy 62.23 60.96) (xy 83.82 60.96)
-		)
-		(stroke
-			(width 0)
-			(type default)
-		)
-	)
-	(wire
-		(pts
-			(xy 49.53 80.01) (xy 52.07 80.01)
-		)
-		(stroke
-			(width 0)
-			(type default)
-		)
-	)
-	(bus
-		(pts
-			(xy 59.69 66.04) (xy 59.69 63.5)
-		)
-		(stroke
-			(width 0)
-			(type default)
-		)
-	)
-	(wire
-		(pts
-			(xy 62.23 63.5) (xy 83.82 63.5)
-		)
-		(stroke
-			(width 0)
-			(type default)
-		)
-	)
-	(label "SCL"
-		(at 63.5 60.96 0)
+			(xy 49.53 81.28) (xy 52.07 81.28)
+		)
+		(stroke
+			(width 0)
+			(type default)
+		)
+	)
+	(wire
+		(pts
+			(xy 125.73 68.58) (xy 120.65 68.58)
+		)
+		(stroke
+			(width 0)
+			(type default)
+		)
+	)
+	(wire
+		(pts
+			(xy 123.19 46.99) (xy 125.73 46.99)
+		)
+		(stroke
+			(width 0)
+			(type default)
+		)
+	)
+	(wire
+		(pts
+			(xy 121.92 66.04) (xy 125.73 66.04)
+		)
+		(stroke
+			(width 0)
+			(type default)
+		)
+	)
+	(wire
+		(pts
+			(xy 123.19 49.53) (xy 125.73 49.53)
+		)
+		(stroke
+			(width 0)
+			(type default)
+		)
+	)
+	(label "GND"
+		(at 123.19 49.53 180)
+		(fields_autoplaced yes)
+		(effects
+			(font
+				(size 1.27 1.27)
+			)
+			(justify right bottom)
+		)
+	)
+	(label "GND"
+		(at 120.65 71.12 0)
 		(fields_autoplaced yes)
 		(effects
@@
 		)
 	)
-	(label "SDA"
-		(at 63.5 63.5 0)
+	(label "+3.3V"
+		(at 121.92 44.45 180)
+		(fields_autoplaced yes)
+		(effects
+			(font
+				(size 1.27 1.27)
+			)
+			(justify right bottom)
+		)
+	)
+	(label "+3.3V"
+		(at 82.55 43.18 0)
 		(fields_autoplaced yes)
 		(effects
@@
 		)
 	)
+	(label "+3.3V"
+		(at 121.92 55.88 180)
+		(fields_autoplaced yes)
+		(effects
+			(font
+				(size 1.27 1.27)
+			)
+			(justify right bottom)
+		)
+	)
 	(label "GND"
-		(at 52.07 80.01 0)
+		(at 52.07 81.28 0)
 		(fields_autoplaced yes)
 		(effects
@@
 		)
 	)
-	(label "GND"
-		(at 82.55 54.61 180)
-		(fields_autoplaced yes)
-		(effects
-			(font
-				(size 1.27 1.27)
-			)
-			(justify right bottom)
+	(hierarchical_label "Direction"
+		(shape output)
+		(at 123.19 46.99 180)
+		(fields_autoplaced yes)
+		(effects
+			(font
+				(size 1.27 1.27)
+			)
+			(justify right)
 		)
 	)
 	(hierarchical_label "GND"
 		(shape passive)
-		(at 49.53 80.01 180)
+		(at 49.53 81.28 180)
+		(fields_autoplaced yes)
+		(effects
+			(font
+				(size 1.27 1.27)
+			)
+			(justify right)
+		)
+	)
+	(hierarchical_label "Water_Level"
+		(shape output)
+		(at 118.11 66.04 180)
 		(fields_autoplaced yes)
 		(effects
@@
 		)
 	)
-	(hierarchical_label "{I2C}"
-		(shape input)
-		(at 58.42 69.85 180)
-		(fields_autoplaced yes)
-		(effects
-			(font
-				(size 1.27 1.27)
-			)
-			(justify right)
-		)
-	)
 	(symbol
-		(lib_id "Device:C")
-		(at 82.55 48.26 0)
+		(lib_id "Device:R")
+		(at 121.92 62.23 0)
 		(unit 1)
 		(exclude_from_sim no)
@@
 		(on_board yes)
 		(dnp no)
-		(property "Reference" "C31"
-			(at 83.82 50.8 0)
+		(property "Reference" "R21"
+			(at 115.824 57.15 0)
 			(effects
 				(font
@@
 				)
 				(justify left)
-				(hide yes)
-			)
-		)
-		(property "Value" "100nF"
-			(at 84.074 45.466 0)
+			)
+		)
+		(property "Value" "100k"
+			(at 121.92 64.008 90)
 			(effects
 				(font
@@
 				)
 				(justify left)
-				(hide yes)
-			)
-		)
-		(property "Footprint" "Capacitor_SMD:C_0603_1608Metric"
-			(at 83.5152 52.07 0)
+			)
+		)
+		(property "Footprint" "Resistor_SMD:R_0603_1608Metric"
+			(at 120.142 62.23 90)
 			(effects
 				(font
@@
 		)
 		(property "Datasheet" "~"
-			(at 82.55 48.26 0)
+			(at 121.92 62.23 0)
 			(effects
 				(font
@@
 		)
 		(property "Description" ""
-			(at 82.55 48.26 0)
+			(at 121.92 62.23 0)
 			(effects
 				(font
@@
 			(project "Weather"
 				(path "/4bc9f80e-0a24-4618-ba5d-3a118070c43e/39e9adaa-0125-4045-bf4e-110370e942be"
-					(reference "C31")
+					(reference "R21")
 					(unit 1)
 				)
@@
 	)
 	(symbol
-		(lib_id "Connector:Screw_Terminal_01x02")
-		(at 130.81 55.88 0)
+		(lib_id "Connector:Screw_Terminal_01x03")
+		(at 130.81 46.99 0)
 		(unit 1)
 		(exclude_from_sim no)
@@
 		(dnp no)
 		(fields_autoplaced yes)
-		(property "Reference" "J31"
-			(at 133.35 55.8799 0)
+		(property "Reference" "J35"
+			(at 133.35 45.7199 0)
 			(effects
 				(font
@@
 			)
 		)
-		(property "Value" "Wind_Direction"
-			(at 133.35 58.4199 0)
+		(property "Value" "Screw_Terminal_01x03"
+			(at 133.35 48.2599 0)
 			(effects
 				(font
@@
 			)
 		)
-		(property "Footprint" "Connector_Phoenix_MSTB:PhoenixContact_MSTBA_2,5_2-G-5,08_1x02_P5.08mm_Horizontal"
-			(at 130.81 55.88 0)
+		(property "Footprint" "Connector_Phoenix_MSTB:PhoenixContact_MSTBA_2,5_3-G-5,08_1x03_P5.08mm_Horizontal"
+			(at 130.81 46.99 0)
 			(effects
 				(font
@@
 		)
 		(property "Datasheet" "~"
-			(at 130.81 55.88 0)
-			(effects
-				(font
-					(size 1.27 1.27)
-				)
-				(hide yes)
-			)
-		)
-		(property "Description" ""
-			(at 130.81 55.88 0)
-			(effects
-				(font
-					(size 1.27 1.27)
-				)
-				(hide yes)
-			)
+			(at 130.81 46.99 0)
+			(effects
+				(font
+					(size 1.27 1.27)
+				)
+				(hide yes)
+			)
+		)
+		(property "Description" "Generic screw terminal, single row, 01x03, script generated (kicad-library-utils/schlib/autogen/connector/)"
+			(at 130.81 46.99 0)
+			(effects
+				(font
+					(size 1.27 1.27)
+				)
+				(hide yes)
+			)
+		)
+		(pin "2"
 		)
 		(pin "1"
 		)
-		(pin "2"
+		(pin "3"
 		)
 		(instances
 			(project "Weather"
 				(path "/4bc9f80e-0a24-4618-ba5d-3a118070c43e/39e9adaa-0125-4045-bf4e-110370e942be"
-					(reference "J31")
+					(reference "J35")
 					(unit 1)
 				)
