File: Projets/Station_meteo/PCB/V0_Prototype/Modules/Power.kicad_sch (KiCad schematic)
At the start: 30 parts, among them J26 Panel, T15 TP, T16 TP, T17 TP, T18 TP, U6 LM317_SOT-223, U7 BL8530

Commit message: Update PCB
Parts:
- added J39: SolderJumper_2_Bridged, Jumper:SolderJumper-2_P1.3mm_Bridged_Pad1.0x1.5mm, symbol Jumper:SolderJumper_2_Bridged
Connections:
- net Vcap: now also J39.2 (B); no longer C13.1, C14.1, C15.1, C16.1, C17.2, D5.1 (K), L5.1, T17.1
- new net: C13.1, C14.1, C15.1, C16.1, C17.2, D5.1 (K), J39.1 (A), L5.1, T17.1
Changed lines of the file:
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@@
-	)
-	(junction
-		(at 129.54 64.77)
-		(diameter 0)
-		(color 0 0 0 0)
 	)
 	(junction
@@
 	(wire
 		(pts
+			(xy 132.08 59.69) (xy 132.08 64.77)
+		)
+		(stroke
+			(width 0)
+			(type default)
+		)
+	)
+	(wire
+		(pts
 			(xy 55.88 64.77) (xy 67.31 64.77)
 		)
@@
 	(wire
 		(pts
-			(xy 129.54 64.77) (xy 132.08 64.77)
-		)
-		(stroke
-			(width 0)
-			(type default)
-		)
-	)
-	(wire
-		(pts
 			(xy 165.1 72.39) (xy 160.02 72.39)
 		)
@@
 	(wire
 		(pts
-			(xy 119.38 64.77) (xy 129.54 64.77)
+			(xy 119.38 64.77) (xy 132.08 64.77)
 		)
 		(stroke
@@
 	(wire
 		(pts
-			(xy 129.54 62.23) (xy 129.54 64.77)
+			(xy 132.08 48.26) (xy 132.08 52.07)
 		)
 		(stroke
@@
 	(hierarchical_label "Vcap"
 		(shape output)
-		(at 129.54 62.23 90)
+		(at 132.08 48.26 90)
 		(fields_autoplaced yes)
 		(effects
@@
 					(unit 1)
 				)
+			)
+		)
+	)
+	(symbol
+		(lib_id "Jumper:SolderJumper_2_Bridged")
+		(at 132.08 55.88 90)
+		(unit 1)
+		(exclude_from_sim yes)
+		(in_bom no)
+		(on_board yes)
+		(dnp no)
+		(fields_autoplaced yes)
+		(property "Reference" "J39"
+			(at 125.73 55.88 0)
+			(effects
+				(font
+					(size 1.27 1.27)
+				)
+				(hide yes)
+			)
+		)
+		(property "Value" "SolderJumper_2_Bridged"
+			(at 128.27 55.88 0)
+			(effects
+				(font
+					(size 1.27 1.27)
+				)
+				(hide yes)
+			)
+		)
+		(property "Footprint" "Jumper:SolderJumper-2_P1.3mm_Bridged_Pad1.0x1.5mm"
+			(at 132.08 55.88 0)
+			(effects
+				(font
+					(size 1.27 1.27)
+				)
+				(hide yes)
+			)
+		)
+		(property "Datasheet" "~"
+			(at 132.08 55.88 0)
+			(effects
+				(font
+					(size 1.27 1.27)
+				)
+				(hide yes)
+			)
+		)
+		(property "Description" "Solder Jumper, 2-pole, closed/bridged"
+			(at 132.08 55.88 0)
+			(effects
+				(font
+					(size 1.27 1.27)
+				)
+				(hide yes)
+			)
+		)
+		(pin "1"
+		)
+		(pin "2"
+		)
+		(instances
+			(project "Weather"
+				(path "/4bc9f80e-0a24-4618-ba5d-3a118070c43e/227f63a5-2f15-4037-8fc8-26de9d1f16ea"
+					(reference "J39")
+					(unit 1)
+				)

Commit message: Add V1 THT version
Parts:
- added D1: SS24, Diode_SMD:D_SMA, symbol Diode:B130-E3
- added J41, J42: Conn_01x01_Pin, Connector_PinHeader_2.54mm:PinHeader_1x01_P2.54mm_Vertical, symbol Connector:Conn_01x01_Pin
- added R38, R39: 100k, Resistor_SMD:R_0603_1608Metric, symbol Device:R
Connections:
- net +3.3V: now also J41.1 (Pin_1)
- net +3.3V_RF: now also J42.1 (Pin_1)
- net +3.3V_Sensors: now also L6.2
- net GND: now also R39.2
- net at C11.2, J26.1 (Pin_1), T15.1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: now also D1.1 (K), R38.1
- new net +5V_USB: D1.2 (A)
- new net V_{panel}: R38.2, R39.1
