File: Projets/Station_meteo/PCB/V0_Prototype/Modules/RTC.kicad_sch (KiCad schematic)
At the start: 6 parts, among them T14 TP, U13 DS3231M

Commit message: Add V1 THT version
Connections:
- net +3.3V: now also U13.4 (~{RST})
- no-connect marks 1 -> 2
Changed lines of the file:
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@@
+	)
+	(no_connect
+		(at 109.22 60.96)
 	)
 	(no_connect
@@
 	(wire
 		(pts
+			(xy 81.28 71.12) (xy 83.82 71.12)
+		)
+		(stroke
+			(width 0)
+			(type default)
+		)
+	)
+	(wire
+		(pts
 			(xy 129.54 48.26) (xy 129.54 50.8)
 		)
@@
 		)
 	)
+	(label "+3.3V"
+		(at 81.28 71.12 180)
+		(fields_autoplaced yes)
+		(effects
+			(font
+				(size 1.27 1.27)
+			)
+			(justify right bottom)
+		)
+	)
