File: Projets/Station_meteo/PCB/V1_THT/Weather.kicad_sch (KiCad schematic)
At the start: 4 parts

Commit message: Update PCB_V1
Other:
- removed sheet GNSS
- removed sheet Interfaces
- removed sheet NRF24
- removed sheet Power
- removed sheet Power_GNSS
- removed sheet Power_RF
- removed sheet Power_Sensors
- removed sheet Programming
- removed sheet RTC
- removed sheet Reset
- removed sheet Temperature
- removed sheet User_Buttons
- removed sheet WIND
- removed sheet XTAL
