File: Projets/Station_meteo/PCB/V1_THT/Shield_Supercapacitors/Modules/MCU.kicad_sch (KiCad schematic)
At the start: 6 parts, among them J1 Conn_02x05_Odd_Even, J2 Conn_02x04_Odd_Even, J3 Conn_02x06_Odd_Even, J4 Conn_02x06_Odd_Even, U1 ATmega328P-P

Commit message: Add shields
Parts:
- renumbered C1 to C2, J1 to J5, J2 to J6, J3 to J7, J4 to J8, U1 to U2
Changed lines of the file:
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@@
 		(on_board yes)
 		(dnp no)
-		(property "Reference" "J3"
+		(property "Reference" "J7"
 			(at 100.076 31.242 0)
 			(effects
@@
 		)
 		(instances
-			(project "Weather"
+			(project "Shield_Supercapacitors"
+				(path "/4bc9f80e-0a24-4618-ba5d-3a118070c43e/e0cfee79-376f-4a95-9177-7f1d98192d82"
+					(reference "J7")
+					(unit 1)
+				)
 				(path "/4bc9f80e-0a24-4618-ba5d-3a118070c43e/6df9e135-6b30-40c1-b1f1-f69b9f79101d"
 					(reference "J3")
-					(unit 1)
-				)
-			)
-			(project "Tracker"
-				(path "/60c5e70b-bc37-4402-aa86-9378cecb8f85/88f718ac-4006-4d52-80c0-50d6cdb3e594"
-					(reference "J20")
 					(unit 1)
 				)
@@
 		(on_board yes)
 		(dnp no)
-		(property "Reference" "J1"
+		(property "Reference" "J5"
 			(at 91.948 53.086 0)
 			(effects
@@
 		)
 		(instances
-			(project "Weather"
+			(project "Shield_Supercapacitors"
+				(path "/4bc9f80e-0a24-4618-ba5d-3a118070c43e/e0cfee79-376f-4a95-9177-7f1d98192d82"
+					(reference "J5")
+					(unit 1)
+				)
 				(path "/4bc9f80e-0a24-4618-ba5d-3a118070c43e/6df9e135-6b30-40c1-b1f1-f69b9f79101d"
 					(reference "J1")
-					(unit 1)
-				)
-			)
-			(project "Tracker"
-				(path "/60c5e70b-bc37-4402-aa86-9378cecb8f85/88f718ac-4006-4d52-80c0-50d6cdb3e594"
-					(reference "J11")
 					(unit 1)
 				)
@@
 		(dnp no)
 		(fields_autoplaced yes)
-		(property "Reference" "U1"
+		(property "Reference" "U2"
 			(at 41.91 25.4314 0)
 			(effects
@@
 		)
 		(instances
-			(project "Weather"
+			(project "Shield_Supercapacitors"
+				(path "/4bc9f80e-0a24-4618-ba5d-3a118070c43e/e0cfee79-376f-4a95-9177-7f1d98192d82"
+					(reference "U2")
+					(unit 1)
+				)
 				(path "/4bc9f80e-0a24-4618-ba5d-3a118070c43e/6df9e135-6b30-40c1-b1f1-f69b9f79101d"
 					(reference "U1")
-					(unit 1)
-				)
-			)
-			(project "Tracker"
-				(path "/60c5e70b-bc37-4402-aa86-9378cecb8f85/88f718ac-4006-4d52-80c0-50d6cdb3e594"
-					(reference "U9")
 					(unit 1)
 				)
@@
 		(dnp no)
 		(fields_autoplaced yes)
-		(property "Reference" "J2"
+		(property "Reference" "J6"
 			(at 100.33 78.74 0)
 			(effects
@@
 		)
 		(instances
-			(project "Weather"
+			(project "Shield_Supercapacitors"
+				(path "/4bc9f80e-0a24-4618-ba5d-3a118070c43e/e0cfee79-376f-4a95-9177-7f1d98192d82"
+					(reference "J6")
+					(unit 1)
+				)
 				(path "/4bc9f80e-0a24-4618-ba5d-3a118070c43e/6df9e135-6b30-40c1-b1f1-f69b9f79101d"
 					(reference "J2")
-					(unit 1)
-				)
-			)
-			(project "Tracker"
-				(path "/60c5e70b-bc37-4402-aa86-9378cecb8f85/88f718ac-4006-4d52-80c0-50d6cdb3e594"
-					(reference "J22")
 					(unit 1)
 				)
@@
 		(on_board yes)
 		(dnp no)
-		(property "Reference" "C1"
+		(property "Reference" "C2"
 			(at 35.052 108.204 90)
 			(effects
@@
 		)
 		(instances
-			(project "Weather"
+			(project "Shield_Supercapacitors"
+				(path "/4bc9f80e-0a24-4618-ba5d-3a118070c43e/e0cfee79-376f-4a95-9177-7f1d98192d82"
+					(reference "C2")
+					(unit 1)
+				)
 				(path "/4bc9f80e-0a24-4618-ba5d-3a118070c43e/6df9e135-6b30-40c1-b1f1-f69b9f79101d"
-					(reference "C1")
-					(unit 1)
-				)
-			)
-			(project "Tracker"
-				(path "/60c5e70b-bc37-4402-aa86-9378cecb8f85/88f718ac-4006-4d52-80c0-50d6cdb3e594"
 					(reference "C1")
 					(unit 1)
@@
 		(on_board yes)
 		(dnp no)
-		(property "Reference" "J4"
+		(property "Reference" "J8"
 			(at 100.33 63.5 0)
 			(effects
@@
 		)
 		(instances
-			(project "Weather"
+			(project "Shield_Supercapacitors"
+				(path "/4bc9f80e-0a24-4618-ba5d-3a118070c43e/e0cfee79-376f-4a95-9177-7f1d98192d82"
+					(reference "J8")
+					(unit 1)
+				)
 				(path "/4bc9f80e-0a24-4618-ba5d-3a118070c43e/6df9e135-6b30-40c1-b1f1-f69b9f79101d"
 					(reference "J4")
 					(unit 1)
 				)
-			)
-			(project "Tracker"
-				(path "/60c5e70b-bc37-4402-aa86-9378cecb8f85/88f718ac-4006-4d52-80c0-50d6cdb3e594"
-					(reference "J12")
-					(unit 1)
-				)
