File: Projets/Station_meteo/PCB/V1_THT/Shield_Supercapacitors/Shield_Lithium.kicad_sch (KiCad schematic)
At the start: 4 parts

Commit message: update of directory
Parts:
- added J1: USB_B_Micro, Connector_USB:USB_Micro-B_Molex-105017-0001, symbol Connector:USB_B_Micro
- added J10: Conn_01x04_Pin, Connector_JST:JST_PH_S4B-PH-K_1x04_P2.00mm_Horizontal, symbol Connector:Conn_01x04_Pin
- added J5: Screw_Terminal_01x03_2.54mm [CREPP], TerminalBlock_Phoenix:TerminalBlock_Phoenix_MKDS-3-3-5.08_1x03_P5.08mm_Horizontal, symbol CREPP_Screw_Terminal:Screw_Terminal_01x03_2.54mm [CREPP]
Connections:
- no-connect marks 7 -> 0
Other:
- removed sheet MCU
- sheet Power ports: added none; removed GND
