File: Projets/Station_meteo/PCB/V1_THT/Base/Modules/User_Buttons.kicad_sch (KiCad schematic)
At the start: 3 parts, among them J7 USR_BTN, SW1 SW_B

Commit message: Update
Parts:
- removed J7: USR_BTN, TerminalBlock_Phoenix:TerminalBlock_Phoenix_MPT-0,5-2-2.54_1x02_P2.54mm_Horizontal, symbol Connector:Conn_01x02_Pin
- removed R10: 10k, Resistor_THT:R_Axial_DIN0207_L6.3mm_D2.5mm_P7.62mm_Horizontal, symbol Device:R
- removed SW1: SW_B, Button_Switch_THT:SW_PUSH_6mm_H8mm, symbol Switch:SW_DPST_x2
- added J30: KF128-2.54_2P, TerminalBlock_Phoenix:TerminalBlock_Phoenix_MPT-0,5-2-2.54_1x02_P2.54mm_Horizontal, symbol Connector:Conn_01x02_Pin
- added R33: 10k, Resistor_SMD:R_0603_1608Metric, symbol Device:R
- added SW2: PB_SMD_12V_50MA_6MM_6MM, Button_Switch_SMD:SW_Push_1P1T_NO_CK_KSC7xxJ, symbol Switch:SW_DPST_x2
Connections:
- net GND: now also J30.1 (Pin_1), SW2.1 (A)
- net VCC: now also R33.1
- new net SELF_TEST: J30.2 (Pin_2), R33.2, SW2.2 (B)
Other:
- title: REset -> User button
Changed lines of the file:
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@@
 	(paper "A5")
 	(title_block
-		(title "REset")
-		(date "2024-04-17")
+		(title "User button")
+		(date "2024-11-03")
 		(rev "1.0")
 	)
@@
 	(label "GND"
 		(at 86.36 72.39 0)
+		(fields_autoplaced yes)
 		(effects
 			(font
@@
 		)
 	)
+	(hierarchical_label "SELF_TEST"
+		(shape bidirectional)
+		(at 74.93 49.53 180)
+		(fields_autoplaced yes)
+		(effects
+			(font
+				(size 1.27 1.27)
+			)
+			(justify right)
+		)
+	)
 	(hierarchical_label "GND"
 		(shape input)
 		(at 64.77 72.39 180)
+		(fields_autoplaced yes)
 		(effects
 			(font
@@
 		)
 	)
-	(hierarchical_label "RESET"
-		(shape bidirectional)
-		(at 74.93 49.53 180)
-		(effects
-			(font
-				(size 1.27 1.27)
-			)
-			(justify right)
-		)
-	)
 	(hierarchical_label "VCC"
 		(shape input)
 		(at 74.93 38.1 180)
+		(fields_autoplaced yes)
 		(effects
 			(font
@@
 		(dnp no)
 		(fields_autoplaced yes)
-		(property "Reference" "SW1"
+		(property "Reference" "SW2"
 			(at 80.01 59.6899 90)
 			(effects
@@
 			)
 		)
-		(property "Value" "SW_B"
+		(property "Value" "PB_SMD_12V_50MA_6MM_6MM"
 			(at 80.01 62.2299 90)
 			(effects
@@
 				)
 				(justify right)
-			)
-		)
-		(property "Footprint" "Button_Switch_THT:SW_PUSH_6mm_H8mm"
+				(hide yes)
+			)
+		)
+		(property "Footprint" "Button_Switch_SMD:SW_Push_1P1T_NO_CK_KSC7xxJ"
 			(at 78.74 60.96 0)
 			(effects
@@
 		(instances
 			(project "Weather"
-				(path "/4bc9f80e-0a24-4618-ba5d-3a118070c43e/f45ab4cc-f222-41d3-b980-a43e09b330cb"
-					(reference "SW1")
-					(unit 1)
-				)
-			)
-			(project "Tracker"
-				(path "/60c5e70b-bc37-4402-aa86-9378cecb8f85/c8bb0d21-4a2a-4279-ac0b-204348079814"
-					(reference "SW4")
-					(unit 1)
-				)
-			)
-		)
-	)
-	(symbol
-		(lib_id "Connector:Conn_01x02_Pin")
-		(at 60.96 58.42 0)
-		(unit 1)
-		(exclude_from_sim no)
-		(in_bom yes)
-		(on_board yes)
-		(dnp no)
-		(property "Reference" "J7"
-			(at 59.69 60.9601 0)
-			(effects
-				(font
-					(size 1.27 1.27)
-				)
-				(justify right)
-			)
-		)
-		(property "Value" "USR_BTN"
-			(at 59.69 58.4201 0)
-			(effects
-				(font
-					(size 1.27 1.27)
-				)
-				(justify right)
-			)
-		)
-		(property "Footprint" "TerminalBlock_Phoenix:TerminalBlock_Phoenix_MPT-0,5-2-2.54_1x02_P2.54mm_Horizontal"
-			(at 60.96 58.42 0)
-			(effects
-				(font
-					(size 1.27 1.27)
-				)
-				(hide yes)
-			)
-		)
-		(property "Datasheet" "~"
-			(at 60.96 58.42 0)
-			(effects
-				(font
-					(size 1.27 1.27)
-				)
-				(hide yes)
-			)
-		)
-		(property "Description" ""
-			(at 60.96 58.42 0)
-			(effects
-				(font
-					(size 1.27 1.27)
-				)
-				(hide yes)
-			)
-		)
-		(pin "1"
-		)
-		(pin "2"
-		)
-		(instances
-			(project "Weather"
-				(path "/4bc9f80e-0a24-4618-ba5d-3a118070c43e/f45ab4cc-f222-41d3-b980-a43e09b330cb"
-					(reference "J7")
-					(unit 1)
-				)
-			)
-			(project "Tracker"
-				(path "/60c5e70b-bc37-4402-aa86-9378cecb8f85/c8bb0d21-4a2a-4279-ac0b-204348079814"
-					(reference "J5")
+				(path "/4bc9f80e-0a24-4618-ba5d-3a118070c43e/ca16450b-3bf0-414c-83a2-71306aba19fe"
+					(reference "SW2")
 					(unit 1)
 				)
@@
 		(dnp no)
 		(fields_autoplaced yes)
-		(property "Reference" "R10"
-			(at 81.28 41.9099 0)
+		(property "Reference" "R33"
+			(at 81.28 41.91 0)
 			(effects
 				(font
@@
 		)
 		(property "Value" "10k"
-			(at 81.28 44.4499 0)
+			(at 81.28 44.45 0)
 			(effects
 				(font
@@
 			)
 		)
-		(property "Footprint" "Resistor_THT:R_Axial_DIN0207_L6.3mm_D2.5mm_P7.62mm_Horizontal"
+		(property "Footprint" "Resistor_SMD:R_0603_1608Metric"
 			(at 76.962 43.18 90)
 			(effects
@@
 		(instances
 			(project "Weather"
-				(path "/4bc9f80e-0a24-4618-ba5d-3a118070c43e/f45ab4cc-f222-41d3-b980-a43e09b330cb"
-					(reference "R13")
+				(path "/4bc9f80e-0a24-4618-ba5d-3a118070c43e/ca16450b-3bf0-414c-83a2-71306aba19fe"
+					(reference "R33")
 					(unit 1)
 				)
 			)
-			(project "Tracker"
-				(path "/60c5e70b-bc37-4402-aa86-9378cecb8f85/c8bb0d21-4a2a-4279-ac0b-204348079814"
-					(reference "R29")
+		)
+	)
+	(symbol
+		(lib_id "Connector:Conn_01x02_Pin")
+		(at 60.96 60.96 0)
+		(mirror x)
+		(unit 1)
+		(exclude_from_sim no)
+		(in_bom yes)
+		(on_board yes)
+		(dnp no)
+		(property "Reference" "J30"
+			(at 59.69 58.4199 0)
+			(effects
+				(font
+					(size 1.27 1.27)
+				)
+				(justify right)
+			)
+		)
+		(property "Value" "KF128-2.54_2P"
+			(at 59.69 60.9599 0)
+			(effects
+				(font
+					(size 1.27 1.27)
+				)
+				(justify right)
+				(hide yes)
+			)
+		)
+		(property "Footprint" "TerminalBlock_Phoenix:TerminalBlock_Phoenix_MPT-0,5-2-2.54_1x02_P2.54mm_Horizontal"
+			(at 60.96 60.96 0)
+			(effects
+				(font
+					(size 1.27 1.27)
+				)
+				(hide yes)
+			)
+		)
+		(property "Datasheet" "~"
+			(at 60.96 60.96 0)
+			(effects
+				(font
+					(size 1.27 1.27)
+				)
+				(hide yes)
+			)
+		)
+		(property "Description" ""
+			(at 60.96 60.96 0)
+			(effects
+				(font
+					(size 1.27 1.27)
+				)
+				(hide yes)
+			)
+		)
+		(pin "1"
+		)
+		(pin "2"
+		)
+		(instances
+			(project "Weather"
+				(path "/4bc9f80e-0a24-4618-ba5d-3a118070c43e/ca16450b-3bf0-414c-83a2-71306aba19fe"
+					(reference "J30")
 					(unit 1)
 				)
