File: Projets/Station_meteo/PCB/V1_THT/Base/Modules/Programming.kicad_sch (KiCad schematic)
At the start: 15 parts, among them J13 USB_C_Receptacle_USB2.0_16P, J14 SolderJumper_2_Bridged, J15 SolderJumper_2_Bridged, J16 SolderJumper_2_Bridged, U10 CH340G, U8 USBLC6-2P6, U9 AMS1117-3.3, Y2 12MHz

Commit message: Update PCB Base
Parts:
- removed C17, C18: 2.2uF, Capacitor_SMD:C_0603_1608Metric, symbol Device:C
- removed D8: LED_USB, LED_SMD:LED_0603_1608Metric, symbol Device:LED
- removed J13: USB_C_Receptacle_USB2.0_16P, Connector_USB:USB_C_Receptacle_GCT_USB4085, symbol Connector:USB_C_Receptacle_USB2.0_16P
- removed J14: SolderJumper_2_Bridged, Jumper:SolderJumper-2_P1.3mm_Bridged_Pad1.0x1.5mm, symbol Jumper:SolderJumper_2_Bridged
- removed R26, R27: 0, Resistor_SMD:R_0603_1608Metric, symbol Device:R
- removed R28: 270, Resistor_SMD:R_0603_1608Metric, symbol PCM_SL_Devices:Resistor_0.5W
- removed U8: USBLC6-2P6, Package_TO_SOT_SMD:SOT-666, symbol Power_Protection:USBLC6-2P6
- removed U9: AMS1117-3.3, Package_TO_SOT_SMD:SOT-223-3_TabPin2, symbol Regulator_Linear:AMS1117-3.3
- added C2: C, symbol Device:C
- added J7: USB_C_Receptacle, CREPP_Connectors_USB:USB_C_Receptacle_GCT_USB4085, symbol CREPP_Connectors_USB_C:USB_C_Receptacle
Connections:
- net +3.3V is gone; now on net +5V: U10.16 (VCC)
- net +5V: now also J7.A4 (VBUS), J7.A9 (VBUS), J7.B4 (VBUS), J7.B9 (VBUS)
- net D+: now also J7.A6 (D+), J7.B6 (D+)
- net D-: now also J7.A7 (D-), J7.B7 (D-)
- net GND: now also C2.2, J7.A1 (GND), J7.A12 (GND), J7.B1 (GND), J7.B12 (GND)
- net at U10.4 (V3): now also C2.1
- no-connect marks 10 -> 19
Other:
- moved on the sheet: C19, U10, Y2

Commit message: Update
Parts:
- renumbered J7 to J8
Changed lines of the file:
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@@
 		(dnp no)
 		(fields_autoplaced yes)
-		(property "Reference" "J7"
+		(property "Reference" "J8"
 			(at 0 19.05 0)
 			(effects
@@
 			(project ""
 				(path "/4bc9f80e-0a24-4618-ba5d-3a118070c43e/d885458e-7b65-4bac-a9ac-9ebb78058802"
-					(reference "J7")
+					(reference "J8")
 					(unit 1)
 				)

Commit message: Update Weather station
Parts:
- Y2: value 12MHz -> Crystal; footprint Crystal:Crystal_SMD_HC49-SD -> Crystal:Crystal_HC49-4H_Vertical
Connections:
- net at U10.7 (XI): now also Y2.2; no longer Y2.1
- net at U10.8 (XO): now also Y2.1; no longer Y2.2
Other:
- moved on the sheet: J8
Changed lines of the file:
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@@
 	)
 	(junction
-		(at 19.05 44.45)
+		(at 48.26 59.69)
 		(diameter 0)
 		(color 0 0 0 0)
 	)
 	(junction
-		(at 19.05 41.91)
+		(at 48.26 57.15)
 		(diameter 0)
 		(color 0 0 0 0)
 	)
 	(no_connect
-		(at 15.24 31.75)
-	)
-	(no_connect
-		(at 15.24 77.47)
-	)
-	(no_connect
-		(at 15.24 54.61)
-	)
-	(no_connect
-		(at 15.24 62.23)
+		(at 44.45 46.99)
+	)
+	(no_connect
+		(at 44.45 92.71)
+	)
+	(no_connect
+		(at 44.45 69.85)
+	)
+	(no_connect
+		(at 44.45 77.47)
 	)
 	(no_connect
@@
 	)
 	(no_connect
-		(at -7.62 92.71)
+		(at 21.59 107.95)
 	)
 	(no_connect
@@
 	)
 	(no_connect
-		(at 15.24 69.85)
+		(at 44.45 85.09)
 	)
 	(no_connect
@@
 	)
 	(no_connect
-		(at 15.24 85.09)
-	)
-	(no_connect
-		(at 15.24 52.07)
-	)
-	(no_connect
-		(at 15.24 67.31)
-	)
-	(no_connect
-		(at 15.24 82.55)
+		(at 44.45 100.33)
+	)
+	(no_connect
+		(at 44.45 67.31)
+	)
+	(no_connect
+		(at 44.45 82.55)
+	)
+	(no_connect
+		(at 44.45 97.79)
 	)
 	(no_connect
@@
 	)
 	(no_connect
-		(at 15.24 74.93)
-	)
-	(no_connect
-		(at 15.24 34.29)
-	)
-	(no_connect
-		(at 15.24 59.69)
+		(at 44.45 90.17)
+	)
+	(no_connect
+		(at 44.45 49.53)
+	)
+	(no_connect
+		(at 44.45 74.93)
 	)
 	(no_connect
@@
 	(wire
 		(pts
-			(xy 15.24 46.99) (xy 19.05 46.99)
+			(xy 44.45 62.23) (xy 48.26 62.23)
 		)
 		(stroke
@@
 	(wire
 		(pts
-			(xy 19.05 44.45) (xy 19.05 46.99)
+			(xy 48.26 59.69) (xy 48.26 62.23)
 		)
 		(stroke
@@
 	(wire
 		(pts
-			(xy 19.05 39.37) (xy 19.05 41.91)
+			(xy 48.26 54.61) (xy 48.26 57.15)
 		)
 		(stroke
@@
 	(wire
 		(pts
-			(xy 19.05 41.91) (xy 21.59 41.91)
-		)
-		(stroke
-			(width 0)
-			(type default)
-		)
-	)
-	(wire
-		(pts
-			(xy 19.05 44.45) (xy 21.59 44.45)
+			(xy 48.26 57.15) (xy 50.8 57.15)
+		)
+		(stroke
+			(width 0)
+			(type default)
+		)
+	)
+	(wire
+		(pts
+			(xy 48.26 59.69) (xy 50.8 59.69)
 		)
 		(stroke
@@
 	(wire
 		(pts
-			(xy 15.24 44.45) (xy 19.05 44.45)
+			(xy 44.45 59.69) (xy 48.26 59.69)
 		)
 		(stroke
@@
 	(wire
 		(pts
-			(xy 15.24 39.37) (xy 19.05 39.37)
+			(xy 44.45 54.61) (xy 48.26 54.61)
 		)
 		(stroke
@@
 	(wire
 		(pts
-			(xy 15.24 26.67) (xy 19.05 26.67)
-		)
-		(stroke
-			(width 0)
-			(type default)
-		)
-	)
-	(wire
-		(pts
-			(xy 15.24 41.91) (xy 19.05 41.91)
-		)
-		(stroke
-			(width 0)
-			(type default)
-		)
-	)
-	(wire
-		(pts
-			(xy 22.86 86.36) (xy 22.86 88.9)
+			(xy 44.45 41.91) (xy 48.26 41.91)
+		)
+		(stroke
+			(width 0)
+			(type default)
+		)
+	)
+	(wire
+		(pts
+			(xy 44.45 57.15) (xy 48.26 57.15)
+		)
+		(stroke
+			(width 0)
+			(type default)
+		)
+	)
+	(wire
+		(pts
+			(xy 52.07 101.6) (xy 52.07 104.14)
 		)
 		(stroke
@@
 	)
 	(label "+5V"
-		(at 15.24 26.67 0)
+		(at 44.45 41.91 0)
 		(effects
 			(font
@@
 	)
 	(label "GND"
-		(at 22.86 86.36 0)
+		(at 52.07 101.6 0)
 		(effects
 			(font
@@
 	)
 	(label "D-"
-		(at 21.59 41.91 0)
+		(at 50.8 57.15 0)
 		(effects
 			(font
@@
 	)
 	(label "GND"
-		(at 0 92.71 0)
+		(at 29.21 107.95 0)
 		(effects
 			(font
@@
 	)
 	(label "D+"
-		(at 21.59 44.45 0)
+		(at 50.8 59.69 0)
 		(effects
 			(font
@@
 	(hierarchical_label "+5V"
 		(shape output)
-		(at 19.05 26.67 0)
+		(at 48.26 41.91 0)
 		(effects
 			(font
@@
 	(hierarchical_label "GND"
 		(shape passive)
-		(at 22.86 88.9 270)
+		(at 52.07 104.14 270)
 		(effects
 			(font
@@
 			)
 			(justify right)
-		)
-	)
-	(symbol
-		(lib_id "Device:Crystal")
-		(at 66.04 76.2 270)
-		(unit 1)
-		(exclude_from_sim no)
-		(in_bom yes)
-		(on_board yes)
-		(dnp no)
-		(fields_autoplaced yes)
-		(property "Reference" "Y2"
-			(at 69.85 74.9299 90)
-			(effects
-				(font
-					(size 1.27 1.27)
-				)
-				(justify left)
-			)
-		)
-		(property "Value" "12MHz"
-			(at 69.85 77.4699 90)
-			(effects
-				(font
-					(size 1.27 1.27)
-				)
-				(justify left)
-			)
-		)
-		(property "Footprint" "Crystal:Crystal_SMD_HC49-SD"
-			(at 66.04 76.2 0)
-			(effects
-				(font
-					(size 1.27 1.27)
-				)
-				(hide yes)
-			)
-		)
-		(property "Datasheet" "~"
-			(at 66.04 76.2 0)
-			(effects
-				(font
-					(size 1.27 1.27)
-				)
-				(hide yes)
-			)
-		)
-		(property "Description" "Two pin crystal"
-			(at 66.04 76.2 0)
-			(effects
-				(font
-					(size 1.27 1.27)
-				)
-				(hide yes)
-			)
-		)
-		(pin "2"
-		)
-		(pin "1"
-		)
-		(instances
-			(project "Weather"
-				(path "/4bc9f80e-0a24-4618-ba5d-3a118070c43e/d885458e-7b65-4bac-a9ac-9ebb78058802"
-					(reference "Y2")
-					(unit 1)
-				)
-			)
 		)
 	)
@@
 	)
 	(symbol
+		(lib_id "Device:Crystal")
+		(at 66.04 76.2 90)
+		(unit 1)
+		(exclude_from_sim no)
+		(in_bom yes)
+		(on_board yes)
+		(dnp no)
+		(fields_autoplaced yes)
+		(property "Reference" "Y2"
+			(at 69.85 74.9299 90)
+			(effects
+				(font
+					(size 1.27 1.27)
+				)
+				(justify right)
+			)
+		)
+		(property "Value" "Crystal"
+			(at 69.85 77.4699 90)
+			(effects
+				(font
+					(size 1.27 1.27)
+				)
+				(justify right)
+			)
+		)
+		(property "Footprint" "Crystal:Crystal_HC49-4H_Vertical"
+			(at 66.04 76.2 0)
+			(effects
+				(font
+					(size 1.27 1.27)
+				)
+				(hide yes)
+			)
+		)
+		(property "Datasheet" "~"
+			(at 66.04 76.2 0)
+			(effects
+				(font
+					(size 1.27 1.27)
+				)
+				(hide yes)
+			)
+		)
+		(property "Description" "Two pin crystal"
+			(at 66.04 76.2 0)
+			(effects
+				(font
+					(size 1.27 1.27)
+				)
+				(hide yes)
+			)
+		)
+		(pin "1"
+		)
+		(pin "2"
+		)
+		(instances
+			(project "Base"
+				(path "/4bc9f80e-0a24-4618-ba5d-3a118070c43e/d885458e-7b65-4bac-a9ac-9ebb78058802"
+					(reference "Y2")
+					(unit 1)
+				)
+			)
+		)
+	)
+	(symbol
 		(lib_id "CREPP_Connectors_USB_C:USB_C_Receptacle")
-		(at 0 52.07 0)
+		(at 29.21 67.31 0)
 		(unit 1)
 		(exclude_from_sim no)
@@
 		(fields_autoplaced yes)
 		(property "Reference" "J8"
-			(at 0 19.05 0)
+			(at 29.21 34.29 0)
 			(effects
 				(font
@@
 		)
 		(property "Value" "USB_C_Receptacle"
-			(at 0 21.59 0)
+			(at 29.21 36.83 0)
 			(effects
 				(font
@@
 		)
 		(property "Footprint" "CREPP_Connectors_USB:USB_C_Receptacle_GCT_USB4085"
-			(at 3.81 52.07 0)
+			(at 33.02 67.31 0)
 			(effects
 				(font
@@
 		)
 		(property "Datasheet" "https://www.usb.org/sites/default/files/documents/usb_type-c.zip"
-			(at 3.81 52.07 0)
+			(at 33.02 67.31 0)
 			(effects
 				(font
@@
 		)
 		(property "Description" "USB Full-Featured Type-C Receptacle connector"
-			(at 0 52.07 0)
-			(effects
-				(font
+			(at 29.21 67.31 0)
+			(effects
+				(font

Commit message: Update
Parts:
- added D2: 1N4148, Diode_THT:D_DO-35_SOD27_P7.62mm_Horizontal, symbol CREPP_Diodes_THT:1N4148
- C19: now left out of the parts list
- C2: value C -> 100nF; footprint (none) -> Capacitor_SMD:C_0603_1608Metric; now left out of the parts list
- Y2: value Crystal -> Crystal HC49-4H 12 MHz
Connections:
- net +5V: now also D2.1 (K), D2.2 (A)
Changed lines of the file:
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@@
 	(wire
 		(pts
-			(xy 44.45 41.91) (xy 48.26 41.91)
+			(xy 44.45 41.91) (xy 60.96 41.91)
 		)
 		(stroke
@@
 	(wire
 		(pts
-			(xy 44.45 57.15) (xy 48.26 57.15)
+			(xy 68.58 41.91) (xy 71.12 41.91)
 		)
 		(stroke
@@
 	(wire
 		(pts
-			(xy 52.07 101.6) (xy 52.07 104.14)
+			(xy 44.45 57.15) (xy 48.26 57.15)
 		)
 		(stroke
@@
 		)
 	)
+	(wire
+		(pts
+			(xy 52.07 101.6) (xy 52.07 104.14)
+		)
+		(stroke
+			(width 0)
+			(type default)
+		)
+	)
 	(label "D+"
 		(at 80.01 62.23 180)
@@
 	(hierarchical_label "+5V"
 		(shape output)
-		(at 48.26 41.91 0)
+		(at 71.12 41.91 0)
 		(effects
 			(font
@@
 	(symbol
 		(lib_id "Device:C")
-		(at 97.79 45.72 90)
-		(unit 1)
-		(exclude_from_sim no)
-		(in_bom yes)
-		(on_board yes)
-		(dnp no)
-		(fields_autoplaced yes)
-		(property "Reference" "C2"
-			(at 97.79 38.1 90)
-			(effects
-				(font
-					(size 1.27 1.27)
-				)
-			)
-		)
-		(property "Value" "C"
-			(at 97.79 40.64 90)
-			(effects
-				(font
-					(size 1.27 1.27)
-				)
-			)
-		)
-		(property "Footprint" ""
-			(at 101.6 44.7548 0)
-			(effects
-				(font
-					(size 1.27 1.27)
-				)
-				(hide yes)
-			)
-		)
-		(property "Datasheet" "~"
-			(at 97.79 45.72 0)
-			(effects
-				(font
-					(size 1.27 1.27)
-				)
-				(hide yes)
-			)
-		)
-		(property "Description" "Unpolarized capacitor"
-			(at 97.79 45.72 0)
-			(effects
-				(font
-					(size 1.27 1.27)
-				)
-				(hide yes)
-			)
-		)
-		(pin "2"
-		)
-		(pin "1"
-		)
-		(instances
-			(project ""
-				(path "/4bc9f80e-0a24-4618-ba5d-3a118070c43e/d885458e-7b65-4bac-a9ac-9ebb78058802"
-					(reference "C2")
-					(unit 1)
-				)
-			)
-		)
-	)
-	(symbol
-		(lib_id "Device:C")
 		(at 113.03 72.39 90)
 		(unit 1)
 		(exclude_from_sim no)
-		(in_bom yes)
+		(in_bom no)
 		(on_board yes)
 		(dnp no)
@@
 				(path "/60c5e70b-bc37-4402-aa86-9378cecb8f85/99b32def-c6e2-4026-bce1-b186caf12b96"
 					(reference "C41")
+					(unit 1)
+				)
+			)
+		)
+	)
+	(symbol
+		(lib_id "Device:C")
+		(at 97.79 45.72 90)
+		(unit 1)
+		(exclude_from_sim no)
+		(in_bom no)
+		(on_board yes)
+		(dnp no)
+		(property "Reference" "C2"
+			(at 94.742 44.45 90)
+			(effects
+				(font
+					(size 1.27 1.27)
+				)
+				(justify left)
+			)
+		)
+		(property "Value" "100nF"
+			(at 106.172 43.434 90)
+			(effects
+				(font
+					(size 1.27 1.27)
+				)
+				(justify left)
+			)
+		)
+		(property "Footprint" "Capacitor_SMD:C_0603_1608Metric"
+			(at 101.6 44.7548 0)
+			(effects
+				(font
+					(size 1.27 1.27)
+				)
+				(hide yes)
+			)
+		)
+		(property "Datasheet" "~"
+			(at 97.79 45.72 0)
+			(effects
+				(font
+					(size 1.27 1.27)
+				)
+				(hide yes)
+			)
+		)
+		(property "Description" ""
+			(at 97.79 45.72 0)
+			(effects
+				(font
+					(size 1.27 1.27)
+				)
+				(hide yes)
+			)
+		)
+		(pin "1"
+		)
+		(pin "2"
+		)
+		(instances
+			(project "Base"
+				(path "/4bc9f80e-0a24-4618-ba5d-3a118070c43e/d885458e-7b65-4bac-a9ac-9ebb78058802"
+					(reference "C2")
 					(unit 1)
 				)
@@
 	)
 	(symbol
+		(lib_id "CREPP_Diodes_THT:1N4148")
+		(at 64.77 41.91 180)
+		(unit 1)
+		(exclude_from_sim no)
+		(in_bom yes)
+		(on_board yes)
+		(dnp no)
+		(fields_autoplaced yes)
+		(property "Reference" "D2"
+			(at 64.77 35.56 0)
+			(effects
+				(font
+					(size 1.27 1.27)
+				)
+			)
+		)
+		(property "Value" "1N4148"
+			(at 64.77 38.1 0)
+			(effects
+				(font
+					(size 1.27 1.27)
+				)
+			)
+		)
+		(property "Footprint" "Diode_THT:D_DO-35_SOD27_P7.62mm_Horizontal"
+			(at 64.77 41.91 0)
+			(effects
+				(font
+					(size 1.27 1.27)
+				)
+				(hide yes)
+			)
+		)
+		(property "Datasheet" "https://assets.nexperia.com/documents/data-sheet/1N4148_1N4448.pdf"
+			(at 64.77 41.91 0)
+			(effects
+				(font
+					(size 1.27 1.27)
+				)
+				(hide yes)
+			)
+		)
+		(property "Description" "100V 0.15A standard switching diode, DO-35"
+			(at 64.77 41.91 0)
+			(effects
+				(font
+					(size 1.27 1.27)
+				)
+				(hide yes)
+			)
+		)
+		(property "Sim.Device" "D"
+			(at 64.77 41.91 0)
+			(effects
+				(font
+					(size 1.27 1.27)
+				)
+				(hide yes)
+			)
+		)
+		(property "Sim.Pins" "1=K 2=A"
+			(at 64.77 41.91 0)
+			(effects
+				(font
+					(size 1.27 1.27)
+				)
+				(hide yes)
+			)
+		)
+		(pin "1"
+		)
+		(pin "2"
+		)
+		(instances
+			(project ""
+				(path "/4bc9f80e-0a24-4618-ba5d-3a118070c43e/d885458e-7b65-4bac-a9ac-9ebb78058802"
+					(reference "D2")
+					(unit 1)
+				)
+			)
+		)
+	)
+	(symbol
 		(lib_id "Jumper:SolderJumper_2_Bridged")
 		(at 109.22 57.15 0)
@@
 		(on_board yes)
 		(dnp no)
-		(fields_autoplaced yes)
 		(property "Reference" "Y2"
 			(at 69.85 74.9299 90)
@@
 			)
 		)
-		(property "Value" "Crystal"
-			(at 69.85 77.4699 90)
+		(property "Value" "Crystal HC49-4H 12 MHz"
+			(at 60.452 83.312 90)
 			(effects
 				(font
@@
 			)
 		)
-		(property "Description" "USB Full-Featured Type-C Receptacle connector"
+		(property "Description" "https://fr.aliexpress.com/item/1005004613618514.html?spm=a2g0o.productlist.main.2.7fd9dEr9dEr9uw&algo_pvid=f74b780a-7363-4b93-ad4a-221d41d593b4&algo_exp_id=f74b780a-7363-4b93-ad4a-221d41d593b4-1&pdp_ext_f=%7B\"order\"%3A\"26\"%2C\"eval\"%3A\"1\"%7D&pdp_npi=4%40dis%21EUR%210.57%210.58%21%21%214.25%214.24%21%40210390b817400918976781972ef217%2112000029834280951%21sea%21FR%210%21ABX&curPageLogUid=7QYJ2519aSGk&utparam-url=scene%3Asearch%7Cquery_from%3A"
 			(at 29.21 67.31 0)
 			(effects

Commit message: Update
Parts:
- removed D2: 1N4148, Diode_THT:D_DO-35_SOD27_P7.62mm_Horizontal, symbol CREPP_Diodes_THT:1N4148
- added D10: 1N5817, Diode_THT:D_DO-41_SOD81_P10.16mm_Horizontal, symbol Diode:1N5817
Connections:
- net +5V: now also D10.1 (K), D10.2 (A)
