File: Projets/Station_meteo/PCB/V1_THT/Base/Modules/RTC.kicad_sch (KiCad schematic)
At the start: 4 parts, among them U3 DS3231M

Commit message: Update
Connections:
- net GND: now also U3.10 (GND), U3.11 (GND), U3.12 (GND), U3.13 (GND), U3.5 (GND), U3.6 (GND), U3.7 (GND), U3.8 (GND), U3.9 (GND)
- net INT: now also U3.3 (~{INT}/SQW)
- net SDA: now reaches R3.1, U3.15 (SDA)
- net SCL: now reaches R12.1, U3.16 (SCL)
- no-connect marks 0 -> 1
Changed lines of the file:
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@@
 		(rev "1.0")
 	)
+	(junction
+		(at 60.96 66.04)
+		(diameter 0)
+		(color 0 0 0 0)
+	)
+	(junction
+		(at 71.12 63.5)
+		(diameter 0)
+		(color 0 0 0 0)
+	)
+	(no_connect
+		(at 107.95 63.5)
+	)
+	(wire
+		(pts
+			(xy 55.88 66.04) (xy 60.96 66.04)
+		)
+		(stroke
+			(width 0)
+			(type default)
+		)
+	)
 	(wire
 		(pts
@@
 	(wire
 		(pts
-			(xy 121.92 50.8) (xy 128.27 50.8)
+			(xy 107.95 71.12) (xy 114.3 71.12)
 		)
 		(stroke
@@
 	(wire
 		(pts
+			(xy 95.25 78.74) (xy 95.25 83.82)
+		)
+		(stroke
+			(width 0)
+			(type default)
+		)
+	)
+	(wire
+		(pts
 			(xy 95.25 53.34) (xy 95.25 58.42)
 		)
@@
 		(pts
 			(xy 82.55 66.04) (xy 60.96 66.04)
+		)
+		(stroke
+			(width 0)
+			(type default)
+		)
+	)
+	(wire
+		(pts
+			(xy 55.88 63.5) (xy 71.12 63.5)
 		)
 		(stroke
@@
 	(global_label "INT"
 		(shape output)
-		(at 128.27 50.8 0)
+		(at 114.3 71.12 0)
 		(fields_autoplaced yes)
 		(effects
@@
 		)
 		(property "Intersheetrefs" "${INTERSHEET_REFS}"
-			(at 134.1581 50.8 0)
+			(at 120.1881 71.12 0)
 			(effects
 				(font
@@
 		)
 	)
+	(hierarchical_label "SDA"
+		(shape bidirectional)
+		(at 55.88 66.04 180)
+		(effects
+			(font
+				(size 1.27 1.27)
+			)
+			(justify right)
+		)
+	)
 	(hierarchical_label "VCC"
 		(shape input)
@@
 		(effects
 			(font
+				(size 1.27 1.27)
+			)
+			(justify right)
+		)
+	)
+	(hierarchical_label "GND"
+		(shape passive)
+		(at 95.25 83.82 270)
+		(effects
+			(font
+				(size 1.27 1.27)
+			)
+			(justify right)
+		)
+	)
+	(hierarchical_label "SCL"
+		(shape bidirectional)
+		(at 55.88 63.5 180)
+		(effects
+			(font

Commit message: Update Weather station
Parts:
- renumbered BT1 to BT2
Changed lines of the file:
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@@
 		(dnp no)
 		(fields_autoplaced yes)
-		(property "Reference" "BT1"
+		(property "Reference" "BT2"
 			(at 101.0285 45.72 90)
 			(effects
@@
 			(project ""
 				(path "/4bc9f80e-0a24-4618-ba5d-3a118070c43e/0d8cecce-0187-4531-a2c2-f9b0d5927047"
-					(reference "BT1")
+					(reference "BT2")
 					(unit 1)
 				)

Commit message: Update
Parts:
- BT2: now left out of the parts list
- R12, R3: value 4.7k -> 10k
Connections:
- net INT renamed WAKE_UP
Changed lines of the file:
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@@
 		(at 107.95 63.5)
 	)
-	(wire
-		(pts
-			(xy 55.88 66.04) (xy 60.96 66.04)
-		)
+	(bus_entry
+		(at 44.45 58.42)
+		(size 2.54 2.54)
+		(stroke
+			(width 0)
+			(type default)
+		)
+	)
+	(bus_entry
+		(at 44.45 63.5)
+		(size 2.54 2.54)
 		(stroke
 			(width 0)
@@
 		)
 	)
+	(bus
+		(pts
+			(xy 44.45 54.61) (xy 44.45 58.42)
+		)
+		(stroke
+			(width 0)
+			(type default)
+		)
+	)
+	(wire
+		(pts
+			(xy 46.99 63.5) (xy 71.12 63.5)
+		)
+		(stroke
+			(width 0)
+			(type default)
+		)
+	)
 	(wire
 		(pts
@@
 	(wire
 		(pts
-			(xy 60.96 66.04) (xy 60.96 58.42)
+			(xy 60.96 66.04) (xy 82.55 66.04)
 		)
 		(stroke
@@
 	(wire
 		(pts
+			(xy 46.99 60.96) (xy 46.99 63.5)
+		)
+		(stroke
+			(width 0)
+			(type default)
+		)
+	)
+	(wire
+		(pts
 			(xy 95.25 78.74) (xy 95.25 83.82)
 		)
@@
 	(wire
 		(pts
-			(xy 82.55 66.04) (xy 60.96 66.04)
-		)
-		(stroke
-			(width 0)
-			(type default)
-		)
-	)
-	(wire
-		(pts
-			(xy 55.88 63.5) (xy 71.12 63.5)
+			(xy 46.99 66.04) (xy 60.96 66.04)
 		)
 		(stroke
@@
 	(wire
 		(pts
+			(xy 60.96 58.42) (xy 60.96 66.04)
+		)
+		(stroke
+			(width 0)
+			(type default)
+		)
+	)
+	(wire
+		(pts
 			(xy 92.71 55.88) (xy 92.71 58.42)
+		)
+		(stroke
+			(width 0)
+			(type default)
+		)
+	)
+	(bus
+		(pts
+			(xy 44.45 58.42) (xy 44.45 63.5)
 		)
 		(stroke
@@
 		)
 	)
+	(label "SCL"
+		(at 49.53 63.5 0)
+		(effects
+			(font
+				(size 1.27 1.27)
+			)
+			(justify left bottom)
+		)
+	)
 	(label "VCC"
 		(at 60.96 48.26 0)
@@
 		)
 	)
+	(label "SDA"
+		(at 49.53 66.04 0)
+		(effects
+			(font
+				(size 1.27 1.27)
+			)
+			(justify left bottom)
+		)
+	)
 	(label "VCC"
 		(at 92.71 55.88 180)
@@
 		)
 	)
-	(global_label "INT"
+	(hierarchical_label "WAKE_UP"
 		(shape output)
 		(at 114.3 71.12 0)
-		(fields_autoplaced yes)
 		(effects
 			(font
@@
 			)
 			(justify left)
-		)
-		(property "Intersheetrefs" "${INTERSHEET_REFS}"
-			(at 120.1881 71.12 0)
-			(effects
-				(font
-					(size 1.27 1.27)
-				)
-				(justify left)
-				(hide yes)
-			)
-		)
-	)
-	(hierarchical_label "SDA"
-		(shape bidirectional)
-		(at 55.88 66.04 180)
-		(effects
-			(font
-				(size 1.27 1.27)
-			)
-			(justify right)
 		)
 	)
@@
 		)
 	)
+	(hierarchical_label "{I2C}"
+		(shape input)
+		(at 44.45 54.61 90)
+		(effects
+			(font
+				(size 1.27 1.27)
+			)
+			(justify left)
+		)
+	)
 	(hierarchical_label "GND"
 		(shape passive)
 		(at 95.25 83.82 270)
-		(effects
-			(font
-				(size 1.27 1.27)
-			)
-			(justify right)
-		)
-	)
-	(hierarchical_label "SCL"
-		(shape bidirectional)
-		(at 55.88 63.5 180)
 		(effects
 			(font
@@
 		(unit 1)
 		(exclude_from_sim no)
-		(in_bom yes)
+		(in_bom no)
 		(on_board yes)
 		(dnp no)
@@
 			)
 		)
-		(property "Value" "4.7k"
+		(property "Value" "10k"
 			(at 63.5 55.8799 0)
 			(effects
@@
 			)
 		)
-		(property "Value" "4.7k"
+		(property "Value" "10k"
 			(at 73.66 55.8799 0)
 			(effects
@@
 			)
 		)
+		(pin "2"
+		)
+		(pin "13"
+		)
 		(pin "9"
 		)
 		(pin "6"
 		)
+		(pin "16"
+		)
+		(pin "4"
+		)
+		(pin "5"
+		)
+		(pin "14"
+		)
+		(pin "3"
+		)
+		(pin "7"
+		)
+		(pin "12"
+		)
+		(pin "11"
+		)
+		(pin "8"
+		)
+		(pin "10"
+		)
+		(pin "1"
+		)
 		(pin "15"
 		)
-		(pin "7"
-		)
-		(pin "3"
-		)
-		(pin "1"
-		)
-		(pin "16"
-		)
-		(pin "2"
-		)
-		(pin "8"
-		)
-		(pin "5"
-		)
-		(pin "4"
-		)
-		(pin "12"
-		)
-		(pin "11"
-		)
-		(pin "10"
-		)
-		(pin "13"
-		)
-		(pin "14"
-		)
 		(instances
-			(project "Base"
+			(project ""
 				(path "/4bc9f80e-0a24-4618-ba5d-3a118070c43e/0d8cecce-0187-4531-a2c2-f9b0d5927047"
 					(reference "U3")
