File: Projets/Station_meteo/PCB/V1_THT/Base/Modules/GNSS.kicad_sch (KiCad schematic)
At the start: 2 parts, among them J11 GNSS_Virtual, J9 Conn_01x04_Socket

Commit message: Update
Parts:
- J11: value GNSS_Virtual -> NEO-6M UBLOX WITH ANTENNA
Connections:
- net +5V: now reaches J9.1 (Pin_1)
- net RX_GNSS: now reaches J9.2 (Pin_2)
- net TX_GNSS: now reaches J9.3 (Pin_3)
- net GND: now reaches J9.4 (Pin_4)
- no-connect marks 0 -> 4
Changed lines of the file:
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@@
 		(rev "1.0")
 	)
-	(wire
-		(pts
-			(xy 40.64 24.13) (xy 43.18 24.13)
-		)
-		(stroke
-			(width 0)
-			(type default)
-		)
-	)
-	(label "VCC"
-		(at 43.18 24.13 0)
-		(effects
-			(font
-				(size 1.27 1.27)
-			)
-			(justify left bottom)
-		)
-	)
-	(hierarchical_label "VCC"
+	(no_connect
+		(at 73.66 68.58)
+	)
+	(no_connect
+		(at 73.66 60.96)
+	)
+	(no_connect
+		(at 73.66 66.04)
+	)
+	(no_connect
+		(at 73.66 63.5)
+	)
+	(wire
+		(pts
+			(xy 66.04 54.61) (xy 74.93 54.61)
+		)
+		(stroke
+			(width 0)
+			(type default)
+		)
+	)
+	(wire
+		(pts
+			(xy 66.04 49.53) (xy 74.93 49.53)
+		)
+		(stroke
+			(width 0)
+			(type default)
+		)
+	)
+	(wire
+		(pts
+			(xy 66.04 57.15) (xy 74.93 57.15)
+		)
+		(stroke
+			(width 0)
+			(type default)
+		)
+	)
+	(wire
+		(pts
+			(xy 66.04 52.07) (xy 74.93 52.07)
+		)
+		(stroke
+			(width 0)
+			(type default)
+		)
+	)
+	(hierarchical_label "+5V"
 		(shape input)
-		(at 40.64 24.13 180)
+		(at 66.04 49.53 180)
+		(effects
+			(font
+				(size 1.27 1.27)
+			)
+			(justify right)
+		)
+	)
+	(hierarchical_label "GND"
+		(shape passive)
+		(at 66.04 57.15 180)
+		(effects
+			(font
+				(size 1.27 1.27)
+			)
+			(justify right)
+		)
+	)
+	(hierarchical_label "RX_GNSS"
+		(shape input)
+		(at 66.04 52.07 180)
+		(effects
+			(font
+				(size 1.27 1.27)
+			)
+			(justify right)
+		)
+	)
+	(hierarchical_label "TX_GNSS"
+		(shape output)
+		(at 66.04 54.61 180)
 		(effects
 			(font
@@
 			)
 		)
-		(property "Value" "GNSS_Virtual"
+		(property "Value" "NEO-6M UBLOX WITH ANTENNA"
 			(at 80.01 66.0399 0)
 			(effects
@@
 			)
 		)
-		(property "Description" "Generic connector, single row, 01x04, script generated"
+		(property "Description" "https://fr.aliexpress.com/item/4001198421663.html?spm=a2g0o.productlist.main.3.19cb20203TUI78&algo_pvid=a54e9259-bcf8-495b-a9e9-95118daa90e9&algo_exp_id=a54e9259-bcf8-495b-a9e9-95118daa90e9-2&pdp_ext_f=%7B\"order\"%3A\"3301\"%2C\"eval\"%3A\"1\"%7D&pdp_npi=4%40dis%21EUR%211.24%210.99%21%21%211.26%211.01%21%40210384b917400921971701493e61da%2110000015275671642%21sea%21FR%210%21ABX&curPageLogUid=ciaQZ1gqdxtb&utparam-url=scene%3Asearch%7Cquery_from%3A"
 			(at 80.01 52.07 0)
 			(effects

Commit message: Update
Changed lines of the file:
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@@
 (kicad_sch
-	(version 20231120)
+	(version 20250114)
 	(generator "eeschema")
-	(generator_version "8.0")
+	(generator_version "9.0")
 	(paper "A5")
 	(title_block

Commit message: Update Schematic
Parts:
- added J12: KF301-5.0-2P, TerminalBlock_Phoenix:TerminalBlock_Phoenix_MKDS-1,5-2_1x02_P5.00mm_Horizontal, symbol Connector:Screw_Terminal_01x02
- added R33: 270, Resistor_THT:R_Axial_DIN0207_L6.3mm_D2.5mm_P7.62mm_Horizontal, symbol Device:R
Connections:
- net +5V: now also R33.1
- net GND: now also J12.2 (Pin_2)
- new net: J12.1 (Pin_1), R33.2
Other:
- note added: "LED Connector"
Changed lines of the file:
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@@
 		(rev "1.0")
+	)
+	(text "LED Connector"
+		(exclude_from_sim no)
+		(at 72.136 26.416 0)
+		(effects
+			(font
+				(size 1.27 1.27)
+			)
+		)
+	)
+	(junction
+		(at 69.85 49.53)
+		(diameter 0)
+		(color 0 0 0 0)
 	)
 	(no_connect
@@
 	(wire
 		(pts
+			(xy 72.39 35.56) (xy 72.39 39.37)
+		)
+		(stroke
+			(width 0)
+			(type default)
+		)
+	)
+	(wire
+		(pts
 			(xy 66.04 54.61) (xy 74.93 54.61)
 		)
@@
 	(wire
 		(pts
-			(xy 66.04 49.53) (xy 74.93 49.53)
+			(xy 69.85 35.56) (xy 69.85 39.37)
+		)
+		(stroke
+			(width 0)
+			(type default)
+		)
+	)
+	(wire
+		(pts
+			(xy 66.04 49.53) (xy 69.85 49.53)
 		)
 		(stroke
@@
 	(wire
 		(pts
+			(xy 69.85 49.53) (xy 74.93 49.53)
+		)
+		(stroke
+			(width 0)
+			(type default)
+		)
+	)
+	(wire
+		(pts
+			(xy 69.85 46.99) (xy 69.85 49.53)
+		)
+		(stroke
+			(width 0)
+			(type default)
+		)
+	)
+	(wire
+		(pts
 			(xy 66.04 52.07) (xy 74.93 52.07)
 		)
@@
 			(width 0)
 			(type default)
+		)
+	)
+	(label "GND"
+		(at 72.39 39.37 0)
+		(effects
+			(font
+				(size 1.27 1.27)
+			)
+			(justify left bottom)
 		)
 	)
@@
 					(unit 1)
 				)
+			)
+		)
+	)
+	(symbol
+		(lib_id "Device:R")
+		(at 69.85 43.18 180)
+		(unit 1)
+		(exclude_from_sim no)
+		(in_bom yes)
+		(on_board yes)
+		(dnp no)
+		(property "Reference" "R33"
+			(at 72.39 41.9099 0)
+			(effects
+				(font
+					(size 1.27 1.27)
+				)
+				(justify right)
+			)
+		)
+		(property "Value" "270"
+			(at 63.5 43.18 0)
+			(effects
+				(font
+					(size 1.27 1.27)
+				)
+				(justify right)
+			)
+		)
+		(property "Footprint" "Resistor_THT:R_Axial_DIN0207_L6.3mm_D2.5mm_P7.62mm_Horizontal"
+			(at 71.628 43.18 90)
+			(effects
+				(font
+					(size 1.27 1.27)
+				)
+				(hide yes)
+			)
+		)
+		(property "Datasheet" "~"
+			(at 69.85 43.18 0)
+			(effects
+				(font
+					(size 1.27 1.27)
+				)
+				(hide yes)
+			)
+		)
+		(property "Description" ""
+			(at 69.85 43.18 0)
+			(effects
+				(font
+					(size 1.27 1.27)
+				)
+				(hide yes)
+			)
+		)
+		(pin "1"
+		)
+		(pin "2"
+		)
+		(instances
+			(project "Base"
+				(path "/4bc9f80e-0a24-4618-ba5d-3a118070c43e/0c209323-0c66-43b8-9e8a-ac76fcff0019"
+					(reference "R33")
+					(unit 1)
+				)
+			)
+		)
+	)
+	(symbol
+		(lib_id "Connector:Screw_Terminal_01x02")
+		(at 69.85 30.48 90)
+		(unit 1)
+		(exclude_from_sim no)
+		(in_bom yes)
+		(on_board yes)
+		(dnp no)
+		(fields_autoplaced yes)
+		(property "Reference" "J12"
+			(at 74.93 29.2099 90)
+			(effects
+				(font
+					(size 1.27 1.27)
+				)
+				(justify right)
+			)
+		)
+		(property "Value" "KF301-5.0-2P"
+			(at 74.93 31.7499 90)
+			(effects
+				(font
+					(size 1.27 1.27)
+				)
+				(justify right)
+			)
+		)
+		(property "Footprint" "TerminalBlock_Phoenix:TerminalBlock_Phoenix_MKDS-1,5-2_1x02_P5.00mm_Horizontal"
+			(at 69.85 30.48 0)
+			(effects
+				(font
+					(size 1.27 1.27)
+				)
+				(hide yes)
+			)
+		)
+		(property "Datasheet" "~"
+			(at 69.85 30.48 0)
+			(effects
+				(font
+					(size 1.27 1.27)
+				)
+				(hide yes)
+			)
+		)
+		(property "Description" "Generic screw terminal, single row, 01x02, script generated (kicad-library-utils/schlib/autogen/connector/)"
+			(at 69.85 30.48 0)
+			(effects
+				(font
+					(size 1.27 1.27)
+				)
+				(hide yes)
+			)
+		)
+		(pin "1"
+		)
+		(pin "2"
+		)
+		(instances
+			(project "Base"
+				(path "/4bc9f80e-0a24-4618-ba5d-3a118070c43e/0c209323-0c66-43b8-9e8a-ac76fcff0019"
+					(reference "J12")
+					(unit 1)
+				)
