File: Projets/Station_meteo/PCB/V1_THT/Base/Modules/OLED.kicad_sch (KiCad schematic)
At the start: 2 parts, among them U3 DS3231M

Commit message: Update Schematic
Parts:
- removed U3: DS3231M, Package_SO:SOIC-16W_7.5x10.3mm_P1.27mm, symbol Timer_RTC:DS3231M
- added R12, R3: 10k, Resistor_THT:R_Axial_DIN0207_L6.3mm_D2.5mm_P7.62mm_Horizontal, symbol Device:R
- added U: DS3231M, Package_SO:SOIC-16W_7.5x10.3mm_P1.27mm, symbol CREPP_RTC:DS3231M
- renumbered BT3 to BT
Connections:
- net GND: now also U.10 (GND), U.11 (GND), U.12 (GND), U.13 (GND), U.5 (GND), U.6 (GND), U.7 (GND), U.8 (GND), U.9 (GND)
- net SCL: now also R12.1, U.16 (SCL)
- net SDA: now also R3.1, U.15 (SDA)
- net VCC: now also R12.2, R3.2, U.2 (VCC), U.4 (~{RST})
- net WAKE_UP: now also U.3 (~{INT}/SQW)
- net at BT.1 (+): now also U.14 (VBAT)
