File: Projets/Station_meteo/PCB/V1_THT/Base/Base.kicad_pcb (KiCad board)
At the start: 2 copper layers, 87.2 x 97.9 mm, 21 parts, among them J1 Conn_02x05_Odd_Even, J10 Conn_01x04_Pin, J2 Conn_02x04_Odd_Even, J3 Conn_02x06_Odd_Even, J4 Conn_02x06_Odd_Even, J5 Screw_Terminal_01x03_2.54mm [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, J6 Screw_Terminal_01x03_2.54mm [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, J7 Screw_Terminal_01x04, J8 Screw_Terminal_01x03_2.54mm [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, J9 Screw_Terminal_01x04, U1 ATmega328P-P, U2 NRF24L01_Breakout, Y1 Crystal

Commit message: Update PCB Base
Parts:
- removed J10: Conn_01x04_Pin, Connector_JST:JST_PH_S4B-PH-K_1x04_P2.00mm_Horizontal
- removed J8: Screw_Terminal_01x03_2.54mm [CREPP], TerminalBlock_Phoenix:TerminalBlock_Phoenix_MKDS-3-3-5.08_1x03_P5.08mm_Horizontal
- removed J9: Screw_Terminal_01x04, TerminalBlock_Phoenix:TerminalBlock_Phoenix_MKDS-3-4-5.08_1x04_P5.08mm_Horizontal
- removed S2, S3, S4: ~, Spacers:Spacer_M3_20mm
- added BT1: Battery_Cell, CREPP_Batteries_holders:MPD_BC501SM-TR, F.Cu at (71.9, 64.0)
- added C19: 100nF, Capacitor_SMD:C_0603_1608Metric, F.Cu at (90.1, 43.6)
- added C3: 100nF, Capacitor_SMD:C_0603_1608Metric, F.Cu at (254.5, 69.7)
- added C4: 100nF, Capacitor_SMD:C_0603_1608Metric, F.Cu at (254.5, 72.2)
- added C5: 100nF, Capacitor_SMD:C_0603_1608Metric, F.Cu at (254.5, 74.8)
- added C6: 100nF, Capacitor_SMD:C_0603_1608Metric, F.Cu at (254.5, 77.3)
- added D1: LED, LED_THT:LED_D3.0mm, F.Cu at (258.2, 77.4)
- added H1: MountingHole_Pad, MountingHole:MountingHole_3.2mm_M3, F.Cu at (267.1, 93.6)
- added J13: JST_Connector, Connector_JST:JST_PH_B4B-PH-K_1x04_P2.00mm_Vertical, F.Cu at (266.1, 85.8)
- added J15: SolderJumper_2_Bridged, Jumper:SolderJumper-2_P1.3mm_Bridged_Pad1.0x1.5mm, F.Cu at (78.7, 37.5)
- added J16: SolderJumper_2_Bridged, Jumper:SolderJumper-2_P1.3mm_Bridged_Pad1.0x1.5mm, F.Cu at (78.6, 42.5)
- added J5: Screw_Terminal_01x02_2.54mm, TerminalBlock_Phoenix:TerminalBlock_Phoenix_MKDS-1,5-2-5.08_1x02_P5.08mm_Horizontal, F.Cu at (256.9, 52.7)
- added J6: Conn_01x03_Pin, Connector_PinHeader_2.54mm:PinHeader_1x03_P2.54mm_Vertical, F.Cu at (255.7, 60.6)
- added JP2: Jumper, Connector_PinHeader_2.54mm:PinHeader_1x02_P2.54mm_Vertical, F.Cu at (263.4, 60.6)
- added JP3: Jumper_2.54mm_blue, CREPP_Jumpers:Jumper_2.54mm_blue, F.Cu at (232.7, 76.6)
- added R10: 10k, Resistor_THT:R_Axial_DIN0207_L6.3mm_D2.5mm_P7.62mm_Horizontal, F.Cu at (232.4, 68.7)
- added R11: 100k, Resistor_THT:R_Axial_DIN0207_L6.3mm_D2.5mm_P7.62mm_Horizontal, F.Cu at (232.4, 72.8)
- added R12: 4.7k, Resistor_THT:R_Axial_DIN0207_L6.3mm_D2.5mm_P7.62mm_Horizontal, F.Cu at (83.3, 59.4)
- added R3: 4.7k, Resistor_THT:R_Axial_DIN0207_L6.3mm_D2.5mm_P7.62mm_Horizontal, F.Cu at (76.8, 76.9)
- added R4: R_10K_SMD_0603, Resistor_SMD:R_0603_1608Metric, F.Cu at (254.5, 79.8)
- added R5: 100k, Resistor_THT:R_Axial_DIN0207_L6.3mm_D2.5mm_P7.62mm_Horizontal, F.Cu at (232.4, 48.5)
- added R6: 10k, Resistor_THT:R_Axial_DIN0207_L6.3mm_D2.5mm_P7.62mm_Horizontal, F.Cu at (232.4, 52.5)
- added R7: 10k, Resistor_THT:R_Axial_DIN0207_L6.3mm_D2.5mm_P7.62mm_Horizontal, F.Cu at (232.4, 56.6)
- added R8: 10k, Resistor_THT:R_Axial_DIN0207_L6.3mm_D2.5mm_P7.62mm_Horizontal, F.Cu at (232.4, 60.6)
- added R9: 270, Resistor_THT:R_Axial_DIN0207_L6.3mm_D2.5mm_P7.62mm_Horizontal, F.Cu at (232.4, 64.7)
- added RV1: R_Potentiometer, Potentiometer_THT:Potentiometer_Bourns_3266Y_Vertical, F.Cu at (263.2, 71.5)
- added S1: ~, CREPP_Spacers:Spacer_M3_MF_05mm, F.Cu at (259.6, 86.6)
- added S5: ~, CREPP_Spacers:Spacer_M3_MF_05mm, F.Cu at (259.6, 93.8)
- added S6: ~, CREPP_Spacers:Spacer_M3_MF_05mm, F.Cu at (259.6, 101.0)
- added S7: ~, CREPP_Spacers:Spacer_M3_MF_05mm, F.Cu at (259.6, 108.2)
- added T10: TP, TestPoint:TestPoint_Pad_D1.0mm, F.Cu at (259.5, 62.9)
- added T11: TP, TestPoint:TestPoint_Pad_D1.0mm, F.Cu at (259.5, 65.9)
- added T9: TP, TestPoint:TestPoint_Pad_D1.0mm, F.Cu at (259.5, 59.8)
- added U10: CH340G, Package_SO:SOIC-16_3.9x9.9mm_P1.27mm, F.Cu at (84.1, 44.3)
- added U3: DS3231M, Package_SO:SOIC-16W_7.5x10.3mm_P1.27mm, F.Cu at (87.6, 68.4)
- added U4: LM358, Package_DIP:DIP-8_W7.62mm, F.Cu at (243.3, 70.6)
- added U5: 74HC123, Package_DIP:DIP-16_W7.62mm_Socket, F.Cu at (243.7, 48.6)
- added Y2: 12MHz, Crystal:Crystal_SMD_HC49-SD, F.Cu at (83.8, 52.8)
- J5: value Screw_Terminal_01x03_2.54mm [CREPP] -> Screw_Terminal_01x02_2.54mm; footprint TerminalBlock_Phoenix:TerminalBlock_Phoenix_MKDS-3-3-5.08_1x03_P5.08mm_Horizontal -> TerminalBlock_Phoenix:TerminalBlock_Phoenix_MKDS-1,5-2-5.08_1x02_P5.08mm_Horizontal
- J6: value Screw_Terminal_01x03_2.54mm [CREPP] -> Conn_01x03_Pin; footprint TerminalBlock_Phoenix:TerminalBlock_Phoenix_MKDS-3-3-5.08_1x03_P5.08mm_Horizontal -> Connector_PinHeader_2.54mm:PinHeader_1x03_P2.54mm_Vertical
- J7: value Screw_Terminal_01x04 -> USB_C_Receptacle; footprint TerminalBlock_Phoenix:TerminalBlock_Phoenix_MKDS-3-4-5.08_1x04_P5.08mm_Horizontal -> CREPP_Connectors_USB:USB_C_Receptacle_GCT_USB4085
- S1: footprint Spacers:Spacer_M3_20mm -> CREPP_Spacers:Spacer_M3_MF_05mm
- moved J7 62.4 mm to (75.3, 42.6)
- moved H4 57.1 mm to (246.4, 126.0)
- moved U2 57.1 mm to (211.2, 100.6)
- moved C1 57.1 mm to (177.3, 57.1)
- moved H3 57.1 mm to (188.4, 126.0)
- moved J6 57.1 mm to (175.3, 116.6)
- moved S1 57.1 mm to (246.2, 38.8)
- moved Y1 57.1 mm to (193.7, 47.4)
- moved J5 57.1 mm to (175.3, 77.8)
- moved H2 57.1 mm to (210.5, 61.5)
- moved J1 55.8 mm to (114.8, 61.9)
- moved J4 53.9 mm to (97.4, 39.0), turned to 0 degrees
- moved J3 47.6 mm to (117.3, 51.7), turned to 180 degrees
- moved J2 38.4 mm to (99.8, 72.1), turned to 180 degrees
- moved U1 30.8 mm to (103.5, 39.0)
Connections:
- J5 pad 1: unconnected-(J5-Pin_1-Pad1) -> Net-(J5-Pin_1)
- J5 pad 2: unconnected-(J5-Pin_2-Pad2) -> Net-(J5-Pin_2)
- J6 pad 1: unconnected-(J6-Pin_1-Pad1) -> Net-(J5-Pin_2)
- J6 pad 2: unconnected-(J6-Pin_2-Pad2) -> /Anemometer1/Anemo_{signal}
- J6 pad 3: unconnected-(J6-Pin_3-Pad3) -> Net-(J5-Pin_1)
Routing:
- removed copper zone on B.Cu, net GND
- removed copper zone on F.Cu, net GND
Other:
- board size 87.2 x 97.9 mm -> 232.8 x 97.6 mm

Commit message: Update
Parts:
- removed U2: NRF24L01_Breakout, RF_Module:nRF24L01_Breakout
- added J8: USB_C_Receptacle, CREPP_Connectors_USB:USB_C_Receptacle_GCT_USB4085, F.Cu at (69.2, 101.2)
- added Q1: FDS4559, Package_SO:SOIC-8_3.9x4.9mm_P1.27mm, F.Cu at (97.0, 103.0)
- added Q2: 2N7002H, Package_TO_SOT_THT:TO-92, F.Cu at (101.3, 90.6)
- added Q3: FDS4559, Package_SO:SOIC-8_3.9x4.9mm_P1.27mm, F.Cu at (103.6, 84.2)
- added Q4: 2N7002H, Package_TO_SOT_THT:TO-92, F.Cu at (94.7, 109.4)
- added R1: 10k, Resistor_SMD:R_0603_1608Metric, F.Cu at (101.2, 107.4)
- added R13: 10k, Resistor_THT:R_Axial_DIN0207_L6.3mm_D2.5mm_P7.62mm_Horizontal, F.Cu at (81.5, 101.6)
- added R2: 100k, Resistor_SMD:R_0603_1608Metric, F.Cu at (101.2, 110.0)
- added R34: 10k, Resistor_SMD:R_0603_1608Metric, F.Cu at (107.8, 88.6)
- added R35: 100k, Resistor_SMD:R_0603_1608Metric, F.Cu at (107.8, 91.2)
- added SW1: SW_B, Button_Switch_THT:SW_PUSH_6mm_H8mm, F.Cu at (82.0, 105.7)
- added U6: AMS1117-3.3, Package_TO_SOT_SMD:SOT-223-3_TabPin2, F.Cu at (71.3, 117.0)
- added U7: NRF24L01_Breakout, RF_Module:nRF24L01_Breakout, F.Cu at (69.1, 83.6)
- J7: value USB_C_Receptacle -> USR_BTN; footprint CREPP_Connectors_USB:USB_C_Receptacle_GCT_USB4085 -> TerminalBlock_Phoenix:TerminalBlock_Phoenix_MPT-0,5-2-2.54_1x02_P2.54mm_Horizontal
- moved Y1 68.8 mm to (125.8, 58.2), turned to 90 degrees
Connections:
- net /Anemometer1/Anemo_{signal} renamed /Anemometer/Anemo_{signal}
- net /Anemometer1/Wind_interrupt renamed /Anemometer/Wind_interrupt
- net Net-(U3-SCL) renamed /RTC/SCL
- net Net-(U3-SDA) renamed /RTC/SDA
- C3 pad 1: /Anemometer1/Vcc -> /Anemometer/+5V
- C5 pad 1: /Anemometer1/Vcc -> /Anemometer/+5V
- R4 pad 1: /Anemometer1/Vcc -> /Anemometer/+5V
- R5 pad 1: /Anemometer1/+5V -> /Anemometer/+5V
- RV1 pad 1: /Anemometer1/Vcc -> /Anemometer/+5V
- U1 pad 10: /MCU/XTAL2/PB7 -> Net-(U1-XTAL2/PB7)
- U1 pad 9: /MCU/XTAL1/PB6 -> Net-(U1-XTAL1/PB6)
- U3 pad 10: Net-(U3-GND-Pad10) -> GND
- U3 pad 11: Net-(U3-GND-Pad10) -> GND
- U3 pad 12: Net-(U3-GND-Pad10) -> GND
- U3 pad 13: Net-(U3-GND-Pad10) -> GND
- U3 pad 3: unconnected-(U3-~{INT}/SQW-Pad3) -> INT
- U3 pad 5: Net-(U3-GND-Pad10) -> GND
- U3 pad 6: Net-(U3-GND-Pad10) -> GND
- U3 pad 7: Net-(U3-GND-Pad10) -> GND
- U3 pad 8: Net-(U3-GND-Pad10) -> GND
- U3 pad 9: Net-(U3-GND-Pad10) -> GND
- U4 pad 8: /Anemometer1/Vcc -> /Anemometer/+5V
- U5 pad 16: /Anemometer1/Vcc -> /Anemometer/+5V
- Y1 pad 1: unconnected-(Y1-Pad1) -> Net-(U1-XTAL2/PB7)
- Y1 pad 2: unconnected-(Y1-Pad2) -> Net-(U1-XTAL1/PB6)

Commit message: Update Weather station
Parts:
- removed BT1: Battery_Cell, CREPP_Batteries_holders:MPD_BC501SM-TR
- removed C3: 100nF, Capacitor_SMD:C_0603_1608Metric
- removed the J5 at (175.3, 77.8)
- removed the J5 at (256.9, 52.7)
- removed the J6 at (255.7, 60.6)
- removed the J6 at (175.3, 116.6)
- removed R34: 10k, Resistor_SMD:R_0603_1608Metric
- removed R35: 100k, Resistor_SMD:R_0603_1608Metric
- removed the S1 at (246.2, 38.8)
- removed the S1 at (259.6, 86.6)
- removed U6: AMS1117-3.3, Package_TO_SOT_SMD:SOT-223-3_TabPin2
- removed U7: NRF24L01_Breakout, RF_Module:nRF24L01_Breakout
- added BT2: Battery_Cell, CREPP_Batteries_holders:MPD_BC501SM-TR, F.Cu at (161.1, 83.4)
- added C11: 10uF, Capacitor_THT:C_Radial_D5.0mm_H11.0mm_P2.00mm, F.Cu at (160.6, 64.7)
- added C8: 10uF, Capacitor_THT:C_Radial_D5.0mm_H11.0mm_P2.00mm, F.Cu at (160.6, 58.2)
- added J10: Screw_Terminal_01x05_5.08mm, TerminalBlock_Phoenix:TerminalBlock_Phoenix_MKDS-1,5-5-5.08_1x05_P5.08mm_Horizontal, F.Cu at (188.2, 61.9)
- added J11: GNSS_Virtual, Connector_PinSocket_2.54mm:PinSocket_1x04_P2.54mm_Vertical, F.Cu at (193.3, 83.6)
- added J5: Screw_Terminal_01x02_2.54mm, TerminalBlock_Phoenix:TerminalBlock_Phoenix_MKDS-1,5-2-5.08_1x02_P5.08mm_Horizontal, F.Cu at (113.3, 44.5)
- added J6: Conn_01x03_Pin, Connector_PinHeader_2.54mm:PinHeader_1x03_P2.54mm_Vertical, F.Cu at (111.1, 62.6)
- added J9: Conn_01x04_Socket, Connector_PinSocket_2.54mm:PinSocket_1x04_P2.54mm_Vertical, F.Cu at (177.6, 40.6)
- added Q10: 2N7000, Package_TO_SOT_THT:TO-92_Inline, F.Cu at (134.8, 66.3)
- added Q5: FDS4559, Package_SO:SOIC-8_3.9x4.9mm_P1.27mm, F.Cu at (145.6, 66.4)
- added Q6: 2N7000, Package_TO_SOT_THT:TO-92_Inline, F.Cu at (151.8, 66.3)
- added Q7: FDS4559, Package_SO:SOIC-8_3.9x4.9mm_P1.27mm, F.Cu at (162.5, 49.7)
- added Q8: 2N7000, Package_TO_SOT_THT:TO-92_Inline, F.Cu at (168.7, 49.6)
- added Q9: 2N7000, Package_TO_SOT_THT:TO-92_Inline, F.Cu at (151.8, 49.6)
- added R14: 10k, Resistor_THT:R_Axial_DIN0207_L6.3mm_D2.5mm_P7.62mm_Horizontal, F.Cu at (126.0, 40.3)
- added R15: 10k, Resistor_THT:R_Axial_DIN0207_L6.3mm_D2.5mm_P7.62mm_Horizontal, F.Cu at (126.0, 44.3)
- added R16: 10k, Resistor_THT:R_Axial_DIN0207_L6.3mm_D2.5mm_P7.62mm_Horizontal, F.Cu at (142.9, 56.9)
- added R17: 10k, Resistor_THT:R_Axial_DIN0207_L6.3mm_D2.5mm_P7.62mm_Horizontal, F.Cu at (142.9, 61.0)
- added R20: 10k, Resistor_THT:R_Axial_DIN0207_L6.3mm_D2.5mm_P7.62mm_Horizontal, F.Cu at (108.9, 116.5)
- added R21: 10k, Resistor_THT:R_Axial_DIN0207_L6.3mm_D2.5mm_P7.62mm_Horizontal, F.Cu at (108.9, 120.5)
- added R22: 10k, Resistor_THT:R_Axial_DIN0207_L6.3mm_D2.5mm_P7.62mm_Horizontal, F.Cu at (152.5, 126.5)
- added R23: 10k, Resistor_THT:R_Axial_DIN0207_L6.3mm_D2.5mm_P7.62mm_Horizontal, F.Cu at (152.5, 130.5)
- added R24: 10k, Resistor_THT:R_Axial_DIN0207_L6.3mm_D2.5mm_P7.62mm_Horizontal, F.Cu at (165.3, 126.5)
- added R25: 10k, Resistor_THT:R_Axial_DIN0207_L6.3mm_D2.5mm_P7.62mm_Horizontal, F.Cu at (165.3, 130.5)
- added R26: 10k, Resistor_THT:R_Axial_DIN0207_L6.3mm_D2.5mm_P7.62mm_Horizontal, F.Cu at (108.9, 126.6)
- added R27: 10k, Resistor_THT:R_Axial_DIN0207_L6.3mm_D2.5mm_P7.62mm_Horizontal, F.Cu at (108.9, 130.6)
- added R30: 10k, Resistor_THT:R_Axial_DIN0207_L6.3mm_D2.5mm_P7.62mm_Horizontal, F.Cu at (159.9, 40.3)
- added R31: 10k, Resistor_THT:R_Axial_DIN0207_L6.3mm_D2.5mm_P7.62mm_Horizontal, F.Cu at (159.9, 44.3)
- added R32: 10k, Resistor_THT:R_Axial_DIN0207_L6.3mm_D2.5mm_P7.62mm_Horizontal, F.Cu at (142.9, 44.3)
- added R33: 10k, Resistor_THT:R_Axial_DIN0207_L6.3mm_D2.5mm_P7.62mm_Horizontal, F.Cu at (126.0, 61.0)
- added S1: ~, CREPP_Spacers:Spacer_M3_MF_05mm, F.Cu at (133.4, 78.7)
- added U2: AMS1117-3.3, Package_TO_SOT_SMD:SOT-223-3_TabPin2, F.Cu at (169.8, 59.1)
- added U8: NRF24L01_Breakout, RF_Module:nRF24L01_Breakout, F.Cu at (153.7, 108.4)
- C1: value 100nF -> 10uF
- C5: value 100nF -> 10uF; footprint Capacitor_SMD:C_0603_1608Metric -> Capacitor_THT:C_Radial_D5.0mm_H11.0mm_P2.00mm
- J13: value JST_Connector -> JST_PH_4P
- Q2: value 2N7002H -> FDS4559; footprint Package_TO_SOT_THT:TO-92 -> Package_SO:SOIC-8_3.9x4.9mm_P1.27mm
- Q4: value 2N7002H -> 2N7000; footprint Package_TO_SOT_THT:TO-92 -> Package_TO_SOT_THT:TO-92_Inline
- R1: footprint Resistor_SMD:R_0603_1608Metric -> Resistor_THT:R_Axial_DIN0207_L6.3mm_D2.5mm_P7.62mm_Horizontal
- R2: value 100k -> 10k; footprint Resistor_SMD:R_0603_1608Metric -> Resistor_THT:R_Axial_DIN0207_L6.3mm_D2.5mm_P7.62mm_Horizontal
- Y2: value 12MHz -> Crystal; footprint Crystal:Crystal_SMD_HC49-SD -> Crystal:Crystal_HC49-4H_Vertical
- moved C5 165.1 mm to (89.4, 69.9)
- moved RV1 147.9 mm to (116.4, 53.1)
- moved T10 144.6 mm to (115.0, 64.9)
- moved T11 144.6 mm to (115.0, 67.9)
- moved T9 144.6 mm to (115.0, 61.8)
- moved JP2 144.6 mm to (118.8, 62.6)
- moved U4 143.9 mm to (99.6, 62.4)
- moved U5 143.9 mm to (100.0, 40.4)
- moved R10 143.9 mm to (88.7, 60.5)
- moved R11 143.9 mm to (88.7, 64.6)
- moved R5 143.9 mm to (88.7, 40.3)
- moved R6 143.9 mm to (88.7, 44.3)
- moved R7 143.9 mm to (88.7, 48.4)
- moved R8 143.9 mm to (88.7, 52.4)
- moved R9 143.9 mm to (88.7, 56.5)
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Connections:
- C1 pad 1: GND -> /MCU/+VCC
- C1 pad 2: /MCU/+VCC -> GND
- J13 pad 1: /VCC -> /+5V
- J7 pad 1: /Reset/RESET -> /MCU/~{RESET}/PC6
- J7 pad 2: /Reset/GND -> GND
- Q1 pad 7: /Power_Handler_Anemo/V_{IN} -> /+5V
- Q1 pad 8: /Power_Handler_Anemo/V_{IN} -> /+5V
- Q2 pad 1: /Power_Handler_RTC/ENABLE -> /NRF24/+3.3V
- Q2 pad 2: GND -> Net-(Q2A-G)
- Q2 pad 3: Net-(Q2-D) -> (no net)
- Q3 pad 2: Net-(Q2-D) -> Net-(Q10-D)
- Q3 pad 7: /Power_Handler_RTC/V_{IN} -> /+5V
- Q3 pad 8: /Power_Handler_RTC/V_{IN} -> /+5V
- Q4 pad 1: /Power_Handler_Anemo/ENABLE -> GND
- Q4 pad 2: GND -> /Power_Handler_NRF24/ENABLE
- Q4 pad 3: Net-(Q1A-G) -> Net-(Q2A-G)
- R1 pad 2: /Power_Handler_Anemo/V_{IN} -> /+5V
- R13 pad 1: /Reset/VCC -> /+5V
- R13 pad 2: /Reset/RESET -> /MCU/~{RESET}/PC6
- R2 pad 1: /Power_Handler_Anemo/ENABLE -> Net-(Q10-D)
- R2 pad 2: GND -> /+5V
- SW1 pad 1: /Reset/GND -> GND
- SW1 pad 2: /Reset/RESET -> /MCU/~{RESET}/PC6
- Y2 pad 1: Net-(U10-XI) -> Net-(U10-XO)
- Y2 pad 2: Net-(U10-XO) -> Net-(U10-XI)
Other:
- board outline removed
