File: Projets/Station_meteo/PCB/V1_THT/Base/Base.kicad_pcb (KiCad board)
At the start: 2 copper layers, 233.5 x 107 mm, 95 parts, among them J1 Conn_02x05_Odd_Even, J10 KF301-5.0-2P, J10 Screw_Terminal_01x05_5.08mm, J11 NEO-6M UBLOX WITH ANTENNA, J12 KF301-5.0-2P, J13 JST_PH_4P, J14 Screw_Terminal_01x02, J15 SolderJumper_2_Bridged, J16 SolderJumper_2_Bridged, J2 Conn_02x04_Odd_Even, J3 Conn_02x06_Odd_Even, J4 Conn_02x06_Odd_Even, J5 Screw_Terminal_01x02_2.54mm, J6 Conn_01x03_Pin, J7 USR_BTN, J8 USB_C_Receptacle, J9 Conn_01x04_Socket, Q1 FDS4559, Q2 FDS4559, Q3 FDS4559, Q4 FDS4559, SW1 SW_B, SW2 SW_B, SW3 SW_B, SW4 SW_B, T10 TP, T11 TP, T9 TP, U1 ATmega328P-P, U10 CH340G, U2 AMS1117-3.3, U3 DS3231M, U4 LM358, U5 74HC123, U6 BME280, U8 NRF24L01_Breakout, Y1 16 MHz HC49-4H, Y2 Crystal HC49-4H 12 MHz

Commit message: Update Base
Parts:
- removed C10: 22pF - disc, Capacitor_THT:C_Radial_D5.0mm_H11.0mm_P2.00mm
- removed the J10 at (200.2, 74.2)
- removed J11: NEO-6M UBLOX WITH ANTENNA, Connector_PinSocket_2.54mm:PinSocket_1x04_P2.54mm_Vertical
- removed SW3: SW_B, Button_Switch_THT:SW_PUSH_6mm_H8mm
- added J17: KF301-5.0-2P, TerminalBlock_Phoenix:TerminalBlock_Phoenix_MKDS-1,5-2_1x02_P5.00mm_Horizontal, F.Cu at (149.3, 86.5)
- added J18: KF301-5.0-2P, TerminalBlock_Phoenix:TerminalBlock_Phoenix_MKDS-1,5-2_1x02_P5.00mm_Horizontal, F.Cu at (149.0, 120.0)
- C2: value C -> 100nF; footprint Capacitor_THT:C_Radial_D5.0mm_H11.0mm_P2.00mm -> Capacitor_SMD:C_0603_1608Metric
- C3: value 100nF -> 22pF - disc; footprint Capacitor_SMD:C_0603_1608Metric -> Capacitor_THT:C_Disc_D4.3mm_W1.9mm_P5.00mm
- C7: footprint Capacitor_THT:C_Disc_D3.0mm_W1.6mm_P2.50mm -> Capacitor_THT:C_Disc_D4.3mm_W1.9mm_P5.00mm
- J14: value Screw_Terminal_01x02 -> KF301-5.0-2P
- J5: value Screw_Terminal_01x02_2.54mm -> KF301-5.0-2P; footprint TerminalBlock_Phoenix:TerminalBlock_Phoenix_MKDS-1,5-2-5.08_1x02_P5.08mm_Horizontal -> TerminalBlock_Phoenix:TerminalBlock_Phoenix_MKDS-1,5-2_1x02_P5.00mm_Horizontal
- moved U6 199.4 mm to (439.3, 100.0)
- moved D4 176.9 mm to (69.0, 130.0)
- moved D5 176.9 mm to (69.0, 133.6)
- moved C7 171.5 mm to (43.0, 103.0), turned to -90 degrees
- moved Q3 154.2 mm to (107.5, 134.0)
- moved R15 154.2 mm to (102.0, 128.0)
- moved R19 154.2 mm to (104.7, 128.4)
- moved C2 154.2 mm to (98.8, 48.0)
- moved Q2 147.4 mm to (87.2, 129.4)
- moved R18 147.4 mm to (84.6, 124.0)
- moved C19 133.6 mm to (51.8, 46.0)
- moved Q1 132.9 mm to (96.6, 88.5)
- moved R2 132.9 mm to (94.0, 83.1)
- moved S1 121.1 mm to (28.0, 61.4)
- moved S5 121.1 mm to (28.0, 68.6)
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Connections:
- C3 pad 1: Net-(U10-V3) -> Net-(U1-XTAL1/PB6)
- C7 pad 1: Net-(U1-XTAL1/PB6) -> Net-(U1-XTAL2/PB7)
- J10 pad 1: unconnected-(J10-Pin_1-Pad1) -> /SCL
- J10 pad 2: unconnected-(J10-Pin_2-Pad2) -> GND
- J12 pad 1: unconnected-(J12-Pin_1-Pad1) -> /Power_Handler_Temperature_Sun/V_{OUT}
- J12 pad 2: unconnected-(J12-Pin_2-Pad2) -> /SDA
- J14 pad 1: Net-(J14-Pin_1) -> unconnected-(J14-Pin_1-Pad1)
- J14 pad 2: Net-(J14-Pin_2) -> unconnected-(J14-Pin_2-Pad2)
- J6 pad 1: Net-(J14-Pin_2) -> Net-(J5-Pin_2)
- J6 pad 3: Net-(J14-Pin_1) -> Net-(J5-Pin_1)
- R11 pad 1: Net-(J14-Pin_1) -> Net-(J5-Pin_1)
- R5 pad 2: Net-(J14-Pin_2) -> Net-(J5-Pin_2)
Other:
- board size 233.5 x 107 mm -> 117.7 x 102.5 mm
