File: Projets/Station_meteo/PCB/V1_THT/Base/Base.kicad_pcb (KiCad board)
At the start: 2 copper layers, 117.7 x 102.5 mm, 94 parts, among them J1 Conn_02x05_Odd_Even, J10 KF301-5.0-2P, J12 KF301-5.0-2P, J13 JST_PH_4P, J14 KF301-5.0-2P, J15 SolderJumper_2_Bridged, J16 SolderJumper_2_Bridged, J17 KF301-5.0-2P, J18 KF301-5.0-2P, J2 Conn_02x04_Odd_Even, J3 Conn_02x06_Odd_Even, J4 Conn_02x06_Odd_Even, J5 KF301-5.0-2P, J6 Conn_01x03_Pin, J7 USR_BTN, J8 USB_C_Receptacle, J9 Conn_01x04_Socket, Q1 FDS4559, Q2 FDS4559, Q3 FDS4559, Q4 FDS4559, SW1 SW_B, SW2 SW_B, SW4 SW_B, T10 TP, T11 TP, T9 TP, U1 ATmega328P-P, U10 CH340G, U2 AMS1117-3.3, U3 DS3231M, U4 LM358, U5 74HC123, U6 BME280, U8 NRF24L01_Breakout, Y1 16 MHz HC49-4H, Y2 Crystal HC49-4H 12 MHz

Commit message: Update Schematic
Parts:
- removed BT2: Battery_Cell, CREPP_Batteries_holders:MPD_BC501SM-TR
- removed D2, D3, D4, D5: 1N4148, Diode_THT:D_DO-35_SOD27_P7.62mm_Horizontal
- removed J10, J14, J17, J18: KF301-5.0-2P, TerminalBlock_Phoenix:TerminalBlock_Phoenix_MKDS-1,5-2_1x02_P5.00mm_Horizontal
- removed J7: USR_BTN, TerminalBlock_Phoenix:TerminalBlock_Phoenix_MPT-0,5-2-2.54_1x02_P2.54mm_Horizontal
- removed J8: USB_C_Receptacle, CREPP_Connectors_USB:USB_C_Receptacle_GCT_USB4085
- removed R12, R3: 10k, Resistor_THT:R_Axial_DIN0207_L6.3mm_D2.5mm_P7.62mm_Horizontal
- removed SW2, SW4: SW_B, Button_Switch_THT:SW_PUSH_6mm_H8mm
- added D10: 1N5817, Diode_THT:D_DO-41_SOD81_P10.16mm_Horizontal, F.Cu at (372.9, 252.1)
- added D7: 1N5817, Diode_THT:D_DO-41_SOD81_P10.16mm_Horizontal, F.Cu at (372.9, 276.6)
- added D8: 1N5817, Diode_THT:D_DO-41_SOD81_P10.16mm_Horizontal, F.Cu at (334.3, 215.4)
- added H5: MountingHole_Pad, MountingHole:MountingHole_3.2mm_M3, F.Cu at (365.1, 253.9)
- added H6: MountingHole_Pad, MountingHole:MountingHole_3.2mm_M3, F.Cu at (365.1, 261.9)
- added J11: NEO-6M UBLOX WITH ANTENNA, Connector_PinSocket_2.54mm:PinSocket_1x04_P2.54mm_Vertical, F.Cu at (352.1, 292.4)
- added J19: Screw_Terminal_01x04, TerminalBlock_Phoenix:TerminalBlock_Phoenix_MKDS-1,5-4-5.08_1x04_P5.08mm_Horizontal, F.Cu at (348.8, 282.2)
- added J20: Screw_Terminal_01x04, TerminalBlock_Phoenix:TerminalBlock_Phoenix_MKDS-1,5-4-5.08_1x04_P5.08mm_Horizontal, F.Cu at (406.8, 258.0)
- added Q5: FDS4559, Package_SO:SOIC-8_3.9x4.9mm_P1.27mm, F.Cu at (375.3, 294.4)
- added Q6: 2N7000, Package_TO_SOT_THT:TO-92_Inline, F.Cu at (390.1, 224.7)
- added Q7: 2N7000, Package_TO_SOT_THT:TO-92_Inline, F.Cu at (377.4, 224.7)
- added R32: 10k, Resistor_THT:R_Axial_DIN0207_L6.3mm_D2.5mm_P7.62mm_Horizontal, F.Cu at (372.6, 280.7)
- added R33: 270, Resistor_THT:R_Axial_DIN0207_L6.3mm_D2.5mm_P7.62mm_Horizontal, F.Cu at (356.0, 304.2)
- added R34: 10k, Resistor_THT:R_Axial_DIN0207_L6.3mm_D2.5mm_P7.62mm_Horizontal, F.Cu at (389.7, 215.3)
- added R35: 10k, Resistor_THT:R_Axial_DIN0207_L6.3mm_D2.5mm_P7.62mm_Horizontal, F.Cu at (389.7, 219.4)
- added R36: 10k, Resistor_THT:R_Axial_DIN0207_L6.3mm_D2.5mm_P7.62mm_Horizontal, F.Cu at (376.9, 215.3)
- added R37: 10k, Resistor_THT:R_Axial_DIN0207_L6.3mm_D2.5mm_P7.62mm_Horizontal, F.Cu at (376.9, 219.4)
- Q1, Q3, Q4: moved to B.Cu
- moved SW1 414.0 mm to (391.5, 294.5)
- moved C19 399.3 mm to (385.9, 264.6)
- moved R13 394.6 mm to (391.1, 290.4), turned to 0 degrees
- moved J16 390.7 mm to (381.7, 266.2)
- moved J15 385.2 mm to (381.7, 262.6)
- moved U10 373.7 mm to (375.3, 266.7)
- moved U3 373.2 mm to (395.9, 280.5), turned to 0 degrees
- moved Y2 371.3 mm to (375.2, 257.5), turned to 0 degrees
- moved H1 370.7 mm to (349.2, 253.9)
- moved R17 361.0 mm to (358.8, 267.9)
- moved C2 358.1 mm to (385.9, 262.1)
- moved J13 356.4 mm to (348.2, 268.6), turned to 0 degrees
- moved R29 355.6 mm to (358.8, 271.9)
- moved R22 353.0 mm to (391.5, 262.1)
- moved C3 346.0 mm to (330.4, 275.7), turned to 0 degrees
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Connections:
- net /Anemometer/+5V renamed /Anemometer-Rain-Wheathervane/+5V
- net /Anemometer/Wind_interrupt renamed /Anemometer-Rain-Wheathervane/Wind_interrupt
- C8 pad 1: /+5V -> Net-(D7-A)
- J12 pad 1: /Power_Handler_Temperature_Sun/V_{OUT} -> Net-(J12-Pin_1)
- J12 pad 2: /SDA -> GND
- J4 pad 11: /Anemometer/Anemo_{signal} -> /MCU/PD4-D4
- J6 pad 2: /Anemometer/Anemo_{signal} -> /Anemometer-Rain-Wheathervane/Anemo_{signal}
- Q4 pad 3: /+5V -> /+3.3V
- R28 pad 1: /+5V -> /+3.3V
- T9 pad 1: /Anemometer/Anemo_{signal} -> /Anemometer-Rain-Wheathervane/Anemo_{signal}
- U2 pad 3: /+5V -> Net-(D7-A)
- U3 pad 4: /+5V -> /RESET
- U5 pad 9: /Anemometer/Anemo_{signal} -> /Anemometer-Rain-Wheathervane/Anemo_{signal}
Routing:
- net /Programming/D-: track 18.8 -> 0.00 mm
- net /MCU/SDA: track 17.9 -> 0.00 mm
- net Net-(U1-XTAL1/PB6): track 17.0 -> 0.00 mm
- net /Programming/D+: track 16.9 -> 0.00 mm
- net Net-(U1-XTAL2/PB7): track 16.0 -> 0.00 mm
- net Net-(BT3-+): track 15.4 -> 0.00 mm
- net Net-(J2-Pin_7): track 7.80 -> 0.00 mm
- net Net-(J2-Pin_3): track 7.80 -> 0.00 mm
- net /MCU/PB0: track 7.80 -> 0.00 mm
- net Net-(J2-Pin_5): track 7.80 -> 0.00 mm
- net Net-(J4-Pin_8): track 7.78 -> 0.00 mm
- net Net-(J4-Pin_4): track 7.78 -> 0.00 mm
- net Net-(J4-Pin_12): track 7.78 -> 0.00 mm
- net Net-(J4-Pin_6): track 7.78 -> 0.00 mm
- net Net-(J4-Pin_2): track 7.78 -> 0.00 mm
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Other:
- board size 117.7 x 102.5 mm -> 158.3 x 257.5 mm
