File: Projets/Station_meteo/PCB/V1_THT/Base/_autosave-Base.kicad_pcb (KiCad board)
At the start: 2 copper layers, 233.5 x 107 mm, 95 parts, among them J1 Conn_02x05_Odd_Even, J10 KF301-5.0-2P, J10 Screw_Terminal_01x05_5.08mm, J11 NEO-6M UBLOX WITH ANTENNA, J12 KF301-5.0-2P, J13 JST_PH_4P, J14 Screw_Terminal_01x02, J15 SolderJumper_2_Bridged, J16 SolderJumper_2_Bridged, J2 Conn_02x04_Odd_Even, J3 Conn_02x06_Odd_Even, J4 Conn_02x06_Odd_Even, J5 Screw_Terminal_01x02_2.54mm, J6 Conn_01x03_Pin, J7 USR_BTN, J8 USB_C_Receptacle, J9 Conn_01x04_Socket, Q1 FDS4559, Q2 FDS4559, Q3 FDS4559, Q4 FDS4559, SW1 SW_B, SW2 SW_B, SW3 SW_B, SW4 SW_B, T10 TP, T11 TP, T9 TP, U1 ATmega328P-P, U10 CH340G, U2 AMS1117-3.3, U3 DS3231M, U4 LM358, U5 74HC123, U6 BME280, U8 NRF24L01_Breakout, Y1 16 MHz HC49-4H, Y2 Crystal HC49-4H 12 MHz

Commit message: Update
Parts:
- removed C7: 22pF - disc, Capacitor_THT:C_Disc_D3.0mm_W1.6mm_P2.50mm
- removed J5: Screw_Terminal_01x02_2.54mm, TerminalBlock_Phoenix:TerminalBlock_Phoenix_MKDS-1,5-2-5.08_1x02_P5.08mm_Horizontal
- C2: value C -> 100nF; footprint Capacitor_THT:C_Radial_D5.0mm_H11.0mm_P2.00mm -> Capacitor_SMD:C_0603_1608Metric
- C3: value 100nF -> 22pF - disc; footprint Capacitor_SMD:C_0603_1608Metric -> Capacitor_THT:C_Radial_D5.0mm_H11.0mm_P2.00mm
- J10: value Screw_Terminal_01x05_5.08mm -> KF301-5.0-2P; footprint TerminalBlock_Phoenix:TerminalBlock_Phoenix_MKDS-1,5-5-5.08_1x05_P5.08mm_Horizontal -> TerminalBlock_Phoenix:TerminalBlock_Phoenix_MKDS-1,5-2_1x02_P5.00mm_Horizontal
Connections:
- C3 pad 1: Net-(U10-V3) -> Net-(U1-XTAL1/PB6)
- J10 pad 1: /Power_Handler_Temperature_Sun/V_{OUT} -> unconnected-(J10-Pin_1-Pad1)
- J10 pad 2: /SDA -> unconnected-(J10-Pin_2-Pad2)
