File: Projets/Station_meteo/PCB/V1_THT/Base/Base2.kicad_pcb (KiCad board)
At the start: 2 copper layers, 117.7 x 102.5 mm, 94 parts, among them J1 Conn_02x05_Odd_Even, J10 KF301-5.0-2P, J12 KF301-5.0-2P, J13 JST_PH_4P, J14 KF301-5.0-2P, J15 SolderJumper_2_Bridged, J16 SolderJumper_2_Bridged, J17 KF301-5.0-2P, J18 KF301-5.0-2P, J2 Conn_02x04_Odd_Even, J3 Conn_02x06_Odd_Even, J4 Conn_02x06_Odd_Even, J5 KF301-5.0-2P, J6 Conn_01x03_Pin, J7 USR_BTN, J8 USB_C_Receptacle, J9 Conn_01x04_Socket, Q1 FDS4559, Q2 FDS4559, Q3 FDS4559, Q4 FDS4559, SW1 SW_B, SW2 SW_B, SW4 SW_B, T10 TP, T11 TP, T9 TP, U1 ATmega328P-P, U10 CH340G, U2 AMS1117-3.3, U3 DS3231M, U4 LM358, U5 74HC123, U6 BME280, U8 NRF24L01_Breakout, Y1 16 MHz HC49-4H, Y2 Crystal HC49-4H 12 MHz

Commit message: Update
Parts:
- removed STACKUP1: , 
- moved U8 12.3 mm to (67.8, 125.6)
- moved R14 6.89 mm to (80.5, 123.3)
- moved S1 2.66 mm to (28.0, 61.4)
Changed lines of the file:
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@@
 	(footprint "CREPP_Spacers:Spacer_M3_MF_05mm"
 		(layer "F.Cu")
-		(at 30.5 60.5)
+		(at 28 61.409462)
 		(property "Reference" "S1"
 			(at 0 -0.5 0)
@@
 		)
 	)
-	(footprint ""
-		(layer "F.Cu")
-		(at 180.5 86)
-		(property "Reference" "STACKUP1"
-			(at 0 0 0)
-			(unlocked yes)
-			(layer "F.SilkS")
-			(hide yes)
-			(effects
-				(font
-					(size 1.5 1.5)
-					(line_spacing 0)
-					(thickness 0.3)
-				)
-			)
-		)
-		(property "Value" ""
-			(at 0 0 0)
-			(unlocked yes)
-			(layer "F.SilkS")
-			(hide yes)
-			(effects
-				(font
-					(size 1.5 1.5)
-					(line_spacing 0)
-					(thickness 0.3)
-				)
-			)
-		)
-		(property "Datasheet" ""
-			(at 0 0 0)
-			(layer "F.Fab")
-			(hide yes)
-			(effects
-				(font
-					(size 1.27 1.27)
-					(thickness 0.15)
-				)
-			)
-		)
-		(property "Description" ""
-			(at 0 0 0)
-			(layer "F.Fab")
-			(hide yes)
-			(effects
-				(font
-					(size 1.27 1.27)
-					(thickness 0.15)
-				)
-			)
-		)
-		(attr board_only exclude_from_pos_files exclude_from_bom)
-		(fp_text user "2"
-			(at 3.042856 0 0)
-			(unlocked yes)
-			(layer "B.Cu")
-			(effects
-				(font
-					(size 1.5 1.5)
-					(line_spacing 0)
-					(thickness 0.3)
-				)
-			)
-		)
-		(embedded_fonts no)
-	)
 	(footprint "Resistor_THT:R_Axial_DIN0207_L6.3mm_D2.5mm_P7.62mm_Horizontal"
 		(layer "F.Cu")
@@
 	(footprint "Resistor_THT:R_Axial_DIN0207_L6.3mm_D2.5mm_P7.62mm_Horizontal"
 		(layer "F.Cu")
-		(at 80.5 130.19 -90)
+		(at 80.55 123.3 -90)
 		(descr "Resistor, Axial_DIN0207 series, Axial, Horizontal, pin pitch=7.62mm, 0.25W = 1/4W, length*diameter=6.3*2.5mm^2, http://cdn-reichelt.de/documents/datenblatt/B400/1_4W%23YAG.pdf")
 		(tags "Resistor Axial_DIN0207 series Axial Horizontal pin pitch 7.62mm 0.25W = 1/4W length 6.3mm diameter 2.5mm")
@@
 	(footprint "RF_Module:nRF24L01_Breakout"
 		(layer "F.Cu")
-		(at 80.04 126.12 180)
+		(at 67.7895 125.62 180)
 		(descr "nRF24L01 breakout board")
 		(tags "nRF24L01 adapter breakout")
@@
 			(layer "F.Cu")
 			(effects
+				(font
+					(size 1.5 1.5)
+					(thickness 0.3)
+				)
+			)
+		)
+	)
+	(dimension
+		(type orthogonal)
+		(layer "F.Cu")
+		(pts
+			(xy 97 121.55) (xy 98.5 0)
+		)
+		(height 83.5)
+		(orientation 1)
+		(format
+			(prefix "")
+			(suffix "")
+			(units 3)
+			(units_format 1)
+			(precision 4)
+		)
+		(style
+			(thickness 0.2)
+			(arrow_length 1.27)
+			(text_position_mode 0)
+			(arrow_direction outward)
+			(extension_height 0.58642)
+			(extension_offset 0.5)
+			(keep_text_aligned yes)
+		)
+		(gr_text "121,5500 mm"
+			(at 178.7 60.775 90)
+			(layer "F.Cu")
+			(effects
